File: pt-module-interface.sch (KiCad schematic (older format))
At the start: 8 parts, among them SW2 SW_Push, SW3 SW_Push

Commit message: Re-annotation
Parts:
- removed D11: LED, symbol LED
- removed R12: 1k8, symbol R
- removed R13: 10k, symbol R
- added D8: LED, symbol LED
- added R10: 1k8, symbol R
- added R9: 10k, symbol R
- renumbered D12 to D9, R14 to R12
Connections:
- net +3V3: now also R9.2
- net GND: now also D8.1 (K)
- net prb1_pwr_btn: now also R9.1; no longer R11.1
- net prb1_pwr_led_in: now also R10.1
- net prb1_rs_btn: now also R11.1
- new net: D8.2 (A), R10.2
Changed lines of the file:
@@
 $EndDescr
 $Comp
-L LED D11
-U 1 1 598198A0
+L LED D8
+U 1 1 59945E53
 P 2600 2500
-AR Path="/59819805/598198A0" Ref="D11"  Part="1"
-AR Path="/598B38EB/598198A0" Ref="D13"  Part="1"
-AR Path="/598B3EA9/598198A0" Ref="D15"  Part="1"
-AR Path="/598B41A3/598198A0" Ref="D17"  Part="1"
-F 0 "D11" H 2600 2600 50  0000 C CNN
+F 0 "D8" H 2600 2600 50  0000 C CNN
 F 1 "LED" H 2600 2400 50  0000 C CNN
 F 2 "" H 2600 2500 50  0001 C CNN
@@
 $Comp
 L SW_Push SW2
-U 1 1 598199D3
+U 1 1 59945E56
 P 2600 3550
-AR Path="/59819805/598199D3" Ref="SW2"  Part="1"
-AR Path="/598B38EB/598199D3" Ref="SW4"  Part="1"
-AR Path="/598B3EA9/598199D3" Ref="SW6"  Part="1"
-AR Path="/598B41A3/598199D3" Ref="SW12"  Part="1"
 F 0 "SW2" H 2650 3650 50  0000 L CNN
 F 1 "SW_Push" H 2600 3490 50  0000 C CNN
@@
 $EndComp
 $Comp
-L R R12
-U 1 1 59819AA1
+L R R10
+U 1 1 59945E5A
 P 3050 2500
-AR Path="/59819805/59819AA1" Ref="R12"  Part="1"
-AR Path="/598B38EB/59819AA1" Ref="R16"  Part="1"
-AR Path="/598B3EA9/59819AA1" Ref="R20"  Part="1"
-AR Path="/598B41A3/59819AA1" Ref="R28"  Part="1"
-F 0 "R12" V 3130 2500 50  0000 C CNN
+F 0 "R10" V 3130 2500 50  0000 C CNN
 F 1 "1k8" V 3050 2500 50  0000 C CNN
 F 2 "" V 2980 2500 50  0001 C CNN
@@
 $EndComp
 $Comp
-L R R11
-U 1 1 5981A7B1
+L R R9
+U 1 1 59945E62
 P 2900 3250
-AR Path="/59819805/5981A7B1" Ref="R11"  Part="1"
-AR Path="/598B38EB/5981A7B1" Ref="R15"  Part="1"
-AR Path="/598B3EA9/5981A7B1" Ref="R19"  Part="1"
-AR Path="/598B41A3/5981A7B1" Ref="R27"  Part="1"
-F 0 "R11" V 2980 3250 50  0000 C CNN
+F 0 "R9" V 2980 3250 50  0000 C CNN
 F 1 "10k" V 2900 3250 50  0000 C CNN
 F 2 "" V 2830 3250 50  0001 C CNN
@@
 $EndComp
 $Comp
-L +3.3V #PWR055
-U 1 1 5981A7F0
+L +3.3V #PWR50
+U 1 1 59945E67
 P 2900 3100
-AR Path="/59819805/5981A7F0" Ref="#PWR055"  Part="1"
-AR Path="/598B38EB/5981A7F0" Ref="#PWR65"  Part="1"
-AR Path="/598B3EA9/5981A7F0" Ref="#PWR71"  Part="1"
-AR Path="/598B41A3/5981A7F0" Ref="#PWR90"  Part="1"
-F 0 "#PWR055" H 2900 2950 50  0001 C CNN
+F 0 "#PWR50" H 2900 2950 50  0001 C CNN
 F 1 "+3.3V" H 2900 3240 50  0000 C CNN
 F 2 "" H 2900 3100 50  0001 C CNN
@@
 $EndComp
 $Comp
-L GND #PWR056
-U 1 1 5981A91C
+L GND #PWR48
+U 1 1 59945E69
 P 2200 3600
-AR Path="/59819805/5981A91C" Ref="#PWR056"  Part="1"
-AR Path="/598B38EB/5981A91C" Ref="#PWR63"  Part="1"
-AR Path="/598B3EA9/5981A91C" Ref="#PWR69"  Part="1"
-AR Path="/598B41A3/5981A91C" Ref="#PWR88"  Part="1"
-F 0 "#PWR056" H 2200 3350 50  0001 C CNN
+F 0 "#PWR48" H 2200 3350 50  0001 C CNN
 F 1 "GND" H 2200 3450 50  0000 C CNN
 F 2 "" H 2200 3600 50  0001 C CNN
@@
 prb1_pwr_btn
 $Comp
-L GND #PWR057
+L GND #PWR49
 U 1 1 5981B0C2
 P 2300 2600
-AR Path="/59819805/5981B0C2" Ref="#PWR057"  Part="1"
-AR Path="/598B38EB/5981B0C2" Ref="#PWR64"  Part="1"
-AR Path="/598B3EA9/5981B0C2" Ref="#PWR70"  Part="1"
-AR Path="/598B41A3/5981B0C2" Ref="#PWR89"  Part="1"
-F 0 "#PWR057" H 2300 2350 50  0001 C CNN
+F 0 "#PWR49" H 2300 2350 50  0001 C CNN
 F 1 "GND" H 2300 2450 50  0000 C CNN
 F 2 "" H 2300 2600 50  0001 C CNN
@@
 U 1 1 59898241
 P 4750 3600
-AR Path="/59819805/59898241" Ref="SW3"  Part="1"
-AR Path="/598B38EB/59898241" Ref="SW5"  Part="1"
-AR Path="/598B3EA9/59898241" Ref="SW7"  Part="1"
-AR Path="/598B41A3/59898241" Ref="SW13"  Part="1"
 F 0 "SW3" H 4800 3700 50  0000 L CNN
 F 1 "SW_Push" H 4750 3540 50  0000 C CNN
@@
 $EndComp
 $Comp
-L R R13
-U 1 1 59898247
+L R R11
+U 1 1 59945E7A
 P 5050 3300
-AR Path="/59819805/59898247" Ref="R13"  Part="1"
-AR Path="/598B38EB/59898247" Ref="R17"  Part="1"
-AR Path="/598B3EA9/59898247" Ref="R21"  Part="1"
-AR Path="/598B41A3/59898247" Ref="R29"  Part="1"
-F 0 "R13" V 5130 3300 50  0000 C CNN
+F 0 "R11" V 5130 3300 50  0000 C CNN
 F 1 "10k" V 5050 3300 50  0000 C CNN
 F 2 "" V 4980 3300 50  0001 C CNN
@@
 $EndComp
 $Comp
-L +3.3V #PWR058
+L +3.3V #PWR53
 U 1 1 5989824D
 P 5050 3150
-AR Path="/59819805/5989824D" Ref="#PWR058"  Part="1"
-AR Path="/598B38EB/5989824D" Ref="#PWR68"  Part="1"
-AR Path="/598B3EA9/5989824D" Ref="#PWR74"  Part="1"
-AR Path="/598B41A3/5989824D" Ref="#PWR93"  Part="1"
-F 0 "#PWR058" H 5050 3000 50  0001 C CNN
+F 0 "#PWR53" H 5050 3000 50  0001 C CNN
 F 1 "+3.3V" H 5050 3290 50  0000 C CNN
 F 2 "" H 5050 3150 50  0001 C CNN
@@
 $EndComp
 $Comp
-L GND #PWR059
-U 1 1 59898253
+L GND #PWR51
+U 1 1 59945E80
 P 4350 3650
-AR Path="/59819805/59898253" Ref="#PWR059"  Part="1"
-AR Path="/598B38EB/59898253" Ref="#PWR66"  Part="1"
-AR Path="/598B3EA9/59898253" Ref="#PWR72"  Part="1"
-AR Path="/598B41A3/59898253" Ref="#PWR91"  Part="1"
-F 0 "#PWR059" H 4350 3400 50  0001 C CNN
+F 0 "#PWR51" H 4350 3400 50  0001 C CNN
 F 1 "GND" H 4350 3500 50  0000 C CNN
 F 2 "" H 4350 3650 50  0001 C CNN
@@
 	5050 3450 5050 3600
 $Comp
-L LED D12
+L LED D9
 U 1 1 598986C7
 P 4900 2500
-AR Path="/59819805/598986C7" Ref="D12"  Part="1"
-AR Path="/598B38EB/598986C7" Ref="D14"  Part="1"
-AR Path="/598B3EA9/598986C7" Ref="D16"  Part="1"
-AR Path="/598B41A3/598986C7" Ref="D18"  Part="1"
-F 0 "D12" H 4900 2600 50  0000 C CNN
+F 0 "D9" H 4900 2600 50  0000 C CNN
 F 1 "LED" H 4900 2400 50  0000 C CNN
 F 2 "" H 4900 2500 50  0001 C CNN
@@
 $EndComp
 $Comp
-L R R14
+L R R12
 U 1 1 598986CD
 P 5350 2500
-AR Path="/59819805/598986CD" Ref="R14"  Part="1"
-AR Path="/598B38EB/598986CD" Ref="R18"  Part="1"
-AR Path="/598B3EA9/598986CD" Ref="R22"  Part="1"
-AR Path="/598B41A3/598986CD" Ref="R30"  Part="1"
-F 0 "R14" V 5430 2500 50  0000 C CNN
+F 0 "R12" V 5430 2500 50  0000 C CNN
 F 1 "1k8" V 5350 2500 50  0000 C CNN
 F 2 "" V 5280 2500 50  0001 C CNN
@@
 $EndComp
 $Comp
-L GND #PWR060
-U 1 1 598986D3
+L GND #PWR52
+U 1 1 59945E8A
 P 4600 2600
-AR Path="/59819805/598986D3" Ref="#PWR060"  Part="1"
-AR Path="/598B38EB/598986D3" Ref="#PWR67"  Part="1"
-AR Path="/598B3EA9/598986D3" Ref="#PWR73"  Part="1"
-AR Path="/598B41A3/598986D3" Ref="#PWR92"  Part="1"
-F 0 "#PWR060" H 4600 2350 50  0001 C CNN
+F 0 "#PWR52" H 4600 2350 50  0001 C CNN
 F 1 "GND" H 4600 2450 50  0000 C CNN
 F 2 "" H 4600 2600 50  0001 C CNN

Commit message: add all the rest of the footprints
Parts:
- D8, D9, SW2, SW3: footprint (none) -> Connectors_Hirose:Hirose_DF13C-02P-1.25V_02x1.25mm_Straight
- R10, R11, R12, R9: footprint (none) -> Resistors_SMD:R_1206_HandSoldering
Changed lines of the file:
@@
 F 0 "D8" H 2600 2600 50  0000 C CNN
 F 1 "LED" H 2600 2400 50  0000 C CNN
-F 2 "" H 2600 2500 50  0001 C CNN
+F 2 "Connectors_Hirose:Hirose_DF13C-02P-1.25V_02x1.25mm_Straight" H 2600 2500 50  0001 C CNN
 F 3 "" H 2600 2500 50  0001 C CNN
 	1    2600 2500
@@
 F 0 "SW2" H 2650 3650 50  0000 L CNN
 F 1 "SW_Push" H 2600 3490 50  0000 C CNN
-F 2 "" H 2600 3750 50  0001 C CNN
+F 2 "Connectors_Hirose:Hirose_DF13C-02P-1.25V_02x1.25mm_Straight" H 2600 3750 50  0001 C CNN
 F 3 "" H 2600 3750 50  0001 C CNN
 	1    2600 3550
@@
 F 0 "R10" V 3130 2500 50  0000 C CNN
 F 1 "1k8" V 3050 2500 50  0000 C CNN
-F 2 "" V 2980 2500 50  0001 C CNN
+F 2 "Resistors_SMD:R_1206_HandSoldering" V 2980 2500 50  0001 C CNN
 F 3 "" H 3050 2500 50  0001 C CNN
 	1    3050 2500
@@
 F 0 "R9" V 2980 3250 50  0000 C CNN
 F 1 "10k" V 2900 3250 50  0000 C CNN
-F 2 "" V 2830 3250 50  0001 C CNN
+F 2 "Resistors_SMD:R_1206_HandSoldering" V 2830 3250 50  0001 C CNN
 F 3 "" H 2900 3250 50  0001 C CNN
 	1    2900 3250
@@
 F 0 "SW3" H 4800 3700 50  0000 L CNN
 F 1 "SW_Push" H 4750 3540 50  0000 C CNN
-F 2 "" H 4750 3800 50  0001 C CNN
+F 2 "Connectors_Hirose:Hirose_DF13C-02P-1.25V_02x1.25mm_Straight" H 4750 3800 50  0001 C CNN
 F 3 "" H 4750 3800 50  0001 C CNN
 	1    4750 3600
@@
 F 0 "R11" V 5130 3300 50  0000 C CNN
 F 1 "10k" V 5050 3300 50  0000 C CNN
-F 2 "" V 4980 3300 50  0001 C CNN
+F 2 "Resistors_SMD:R_1206_HandSoldering" V 4980 3300 50  0001 C CNN
 F 3 "" H 5050 3300 50  0001 C CNN
 	1    5050 3300
@@
 F 0 "D9" H 4900 2600 50  0000 C CNN
 F 1 "LED" H 4900 2400 50  0000 C CNN
-F 2 "" H 4900 2500 50  0001 C CNN
+F 2 "Connectors_Hirose:Hirose_DF13C-02P-1.25V_02x1.25mm_Straight" H 4900 2500 50  0001 C CNN
 F 3 "" H 4900 2500 50  0001 C CNN
 	1    4900 2500
@@
 F 0 "R12" V 5430 2500 50  0000 C CNN
 F 1 "1k8" V 5350 2500 50  0000 C CNN
-F 2 "" V 5280 2500 50  0001 C CNN
+F 2 "Resistors_SMD:R_1206_HandSoldering" V 5280 2500 50  0001 C CNN
 F 3 "" H 5350 2500 50  0001 C CNN
 	1    5350 2500
