File: pt-module-mcu.sch (KiCad schematic (older format))
At the start: 12 parts

Commit message: I made a connect
Parts:
- added 10k?: R, symbol R
- added SW?: SW_Push, symbol SW_Push
Connections:
- net +3V3: now also SW?.1
- net BUS_TERM_CTRL: now also U?.36 (ADC2_IN15/COMP6_INM/HRTIM1_CHD2/RTC_REFIN/TIM15_CH1N/TIM15_CH2/TIM1_CH3N/PB15); no longer U?.8 (PC0/ADC1_IN6/ADC2_IN6/TIM1_CH1)
- net GND: now also U?.12 (VSSA), U?.18 (VSS), U?.31 (VSS), U?.47 (VSS), U?.63 (VSS), 10k?.1
- net prb_LED_1_pwr: now reaches U?.10 (PC2/ADC1_IN8/ADC2_IN8/TIM1_CH3)
- net prb_LED_1_rs: now reaches U?.11 (PC3/ADC1_IN9/ADC2_IN9/TIM1_BKIN2/TIM1_CH4)
- net prb_btn_4_rs: now reaches U?.2 (PC13/RTC_OUT_ALARM/RTC_OUT_CALIB/RTC_TAMP1/RTC_TS/SYS_WKUP2/TIM1_CH1N)
- net prb_btn_pwr_master: now reaches U?.20 (ADC2_IN1/COMP2_INM/COMP4_INM/COMP6_INM/DAC1_OUT1/SPI1_NSS/TIM3_CH2/TSC_G2_IO1/USART2_CK/PA4)
- net prb_btn_rs_master: now reaches U?.21 (ADC2_IN2/DAC1_OUT2/OPAMP2_VINM/OPAMP2_VINM_SEC/SPI1_SCK/TIM2_CH1/TIM2_ETR/TSC_G2_IO2/PA5)
- net prb_btn_2_pwr: now reaches U?.24 (PC4/ADC2_IN5/TIM1_ETR/USART1_TX)
- net prb_btn_2_rs: now reaches U?.25 (PC5/ADC2_IN11/OPAMP2_VINM/OPAMP2_VINM_SEC/TIM15_BKIN/TSC_G3_IO1/USART1_RX)
- net prb_LED_4_pwr: now reaches U?.3 (PC14/RCC_OSC32_IN)
- net prb_LED_2_pwr: now reaches U?.37 (PC6/COMP6_OUT/HRTIM1_EEV10/TIM3_CH1)
- net prb_LED_2_rs: now reaches U?.38 (PC7/HRTIM1_FLT5/TIM3_CH2)
- net prb_btn_3_pwr: now reaches U?.39 (PC8/HRTIM1_CHE1/TIM3_CH3)
- net prb_LED_4_rs: now reaches U?.4 (PC15/RCC_OSC32_OUT)
- net prb_btn_3_rs: now reaches U?.40 (PC9/DAC1_EXTI9/DAC2_EXTI9/HRTIM1_CHE2/TIM3_CH4)
- net prb_LED_3_pwr: now reaches U?.51 (PC10/USART3_TX)
- net prb_LED_3_rs: now reaches U?.52 (PC11/HRTIM1_EEV2/USART3_RX)
- net prb_btn_4_pwr: now reaches U?.53 (PC12/HRTIM1_EEV1/USART3_CK)
- net at U?.60 (BOOT0): now also 10k?.2, SW?.2
- net prb_btn_1_rs: now reaches U?.9 (PC1/ADC1_IN7/ADC2_IN7/TIM1_CH2)
- new net prb_btn_1_pwr: U?.8 (PC0/ADC1_IN6/ADC2_IN6/TIM1_CH1)
Other:
- moved on the sheet: 16Mhz, 27pF
Changed lines of the file:
@@
 L Crystal 16Mhz
 U 1 1 597ECED5
-P 1850 6100
-F 0 "16Mhz" H 1850 6250 50  0000 C CNN
-F 1 "Crystal" H 1850 5950 50  0000 C CNN
-F 2 "" H 1850 6100 50  0001 C CNN
-F 3 "" H 1850 6100 50  0001 C CNN
-	1    1850 6100
+P 1500 6400
+F 0 "16Mhz" H 1500 6550 50  0000 C CNN
+F 1 "Crystal" H 1500 6250 50  0000 C CNN
+F 2 "" H 1500 6400 50  0001 C CNN
+F 3 "" H 1500 6400 50  0001 C CNN
+	1    1500 6400
 	1    0    0    -1
 $EndComp
@@
 L C_Small 27pF
 U 1 1 597ECFD6
-P 1500 6300
-F 0 "27pF" H 1510 6370 50  0000 L CNN
-F 1 "C_Small" H 1510 6220 50  0000 L CNN
-F 2 "" H 1500 6300 50  0001 C CNN
-F 3 "" H 1500 6300 50  0001 C CNN
-	1    1500 6300
+P 1150 6600
+F 0 "27pF" H 1160 6670 50  0000 L CNN
+F 1 "C_Small" H 1160 6520 50  0000 L CNN
+F 2 "" H 1150 6600 50  0001 C CNN
+F 3 "" H 1150 6600 50  0001 C CNN
+	1    1150 6600
 	1    0    0    -1
 $EndComp
@@
 L C_Small 27pF
 U 1 1 597ED20D
-P 2200 6300
-F 0 "27pF" H 2210 6370 50  0000 L CNN
-F 1 "C_Small" H 2210 6220 50  0000 L CNN
-F 2 "" H 2200 6300 50  0001 C CNN
-F 3 "" H 2200 6300 50  0001 C CNN
-	1    2200 6300
-	1    0    0    -1
-$EndComp
-$Comp
-L GND #PWR016
+P 1850 6600
+F 0 "27pF" H 1860 6670 50  0000 L CNN
+F 1 "C_Small" H 1860 6520 50  0000 L CNN
+F 2 "" H 1850 6600 50  0001 C CNN
+F 3 "" H 1850 6600 50  0001 C CNN
+	1    1850 6600
+	1    0    0    -1
+$EndComp
+$Comp
+L GND #PWR031
 U 1 1 597EDE48
-P 1500 6500
-F 0 "#PWR016" H 1500 6250 50  0001 C CNN
-F 1 "GND" H 1500 6350 50  0000 C CNN
-F 2 "" H 1500 6500 50  0001 C CNN
-F 3 "" H 1500 6500 50  0001 C CNN
-	1    1500 6500
-	1    0    0    -1
-$EndComp
-$Comp
-L GND #PWR017
+P 1150 6800
+F 0 "#PWR031" H 1150 6550 50  0001 C CNN
+F 1 "GND" H 1150 6650 50  0000 C CNN
+F 2 "" H 1150 6800 50  0001 C CNN
+F 3 "" H 1150 6800 50  0001 C CNN
+	1    1150 6800
+	1    0    0    -1
+$EndComp
+$Comp
+L GND #PWR032
 U 1 1 597EDE64
-P 2200 6500
-F 0 "#PWR017" H 2200 6250 50  0001 C CNN
-F 1 "GND" H 2200 6350 50  0000 C CNN
-F 2 "" H 2200 6500 50  0001 C CNN
-F 3 "" H 2200 6500 50  0001 C CNN
-	1    2200 6500
-	1    0    0    -1
-$EndComp
-Text Label 2200 5950 1    60   ~ 0
+P 1850 6800
+F 0 "#PWR032" H 1850 6550 50  0001 C CNN
+F 1 "GND" H 1850 6650 50  0000 C CNN
+F 2 "" H 1850 6800 50  0001 C CNN
+F 3 "" H 1850 6800 50  0001 C CNN
+	1    1850 6800
+	1    0    0    -1
+$EndComp
+Text Label 1850 6250 1    60   ~ 0
 RCC_OSC_OUT
-Text Label 1500 5950 1    60   ~ 0
+Text Label 1150 6250 1    60   ~ 0
 RCC_OSC_IN
 $Comp
@@
 $EndComp
 $Comp
-L GND #PWR019
+L GND #PWR033
 U 1 1 597EF838
 P 1750 1850
-F 0 "#PWR019" H 1750 1600 50  0001 C CNN
+F 0 "#PWR033" H 1750 1600 50  0001 C CNN
 F 1 "GND" H 1750 1700 50  0000 C CNN
 F 2 "" H 1750 1850 50  0001 C CNN
@@
 $EndComp
 $Comp
-L GND #PWR020
+L GND #PWR034
 U 1 1 597F238E
-P 5800 900
-F 0 "#PWR020" H 5800 650 50  0001 C CNN
-F 1 "GND" H 5800 750 50  0000 C CNN
-F 2 "" H 5800 900 50  0001 C CNN
-F 3 "" H 5800 900 50  0001 C CNN
-	1    5800 900
-	-1   0    0    1
+P 5400 1050
+F 0 "#PWR034" H 5400 800 50  0001 C CNN
+F 1 "GND" H 5400 900 50  0000 C CNN
+F 2 "" H 5400 1050 50  0001 C CNN
+F 3 "" H 5400 1050 50  0001 C CNN
+	1    5400 1050
+	1    0    0    -1
 $EndComp
 Text Label 2550 3250 2    60   ~ 0
@@
 NoConn ~ 2550 2450
 $Comp
-L +3.3V #PWR023
+L +3.3V #PWR035
 U 1 1 5980C7A4
 P 5900 1650
-F 0 "#PWR023" H 5900 1500 50  0001 C CNN
+F 0 "#PWR035" H 5900 1500 50  0001 C CNN
 F 1 "+3.3V" H 5900 1790 50  0000 C CNN
 F 2 "" H 5900 1650 50  0001 C CNN
@@
 $EndComp
 $Comp
-L +3.3V #PWR024
+L +3.3V #PWR036
 U 1 1 5980CC21
 P 1750 2050
-F 0 "#PWR024" H 1750 1900 50  0001 C CNN
+F 0 "#PWR036" H 1750 1900 50  0001 C CNN
 F 1 "+3.3V" H 1750 2190 50  0000 C CNN
 F 2 "" H 1750 2050 50  0001 C CNN
@@
 Wire Wire Line
 	2200 2050 2550 2050
-Connection ~ 2200 6100
-Connection ~ 1500 6100
-Wire Wire Line
-	1500 6400 1500 6500
-Wire Wire Line
-	2200 6400 2200 6500
-Wire Wire Line
-	1500 5950 1500 6200
-Wire Wire Line
-	1700 6100 1500 6100
-Wire Wire Line
-	2200 5950 2200 6200
-Wire Wire Line
-	2000 6100 2200 6100
+Connection ~ 1850 6400
+Connection ~ 1150 6400
+Wire Wire Line
+	1150 6700 1150 6800
+Wire Wire Line
+	1850 6700 1850 6800
+Wire Wire Line
+	1150 6250 1150 6500
+Wire Wire Line
+	1350 6400 1150 6400
+Wire Wire Line
+	1850 6250 1850 6500
+Wire Wire Line
+	1650 6400 1850 6400
 Wire Wire Line
 	5900 1650 6800 1650
@@
 Connection ~ 6350 1650
 Wire Wire Line
-	6800 1650 6800 1200
+	6800 1200 6800 1650
 Connection ~ 6450 1650
 Wire Wire Line
-	6800 1200 5800 1200
+	5800 1200 6800 1200
 Connection ~ 6600 1200
 Connection ~ 6400 1200
@@
 Connection ~ 6000 1200
 Wire Wire Line
-	5800 1000 6800 1000
+	5400 1000 6800 1000
 Connection ~ 6000 1000
 Connection ~ 6600 1000
 Connection ~ 6200 1000
 Connection ~ 6400 1000
-Wire Wire Line
-	5800 1000 5800 900
 Connection ~ 5800 1000
 Connection ~ 6800 1200
@@
 Text HLabel 9950 2150 2    60   Output ~ 0
 UART2_de
+Text HLabel 9950 5250 2    60   Input ~ 0
+BUS_TERM_CTRL
+$Comp
+L R 10k?
+U 1 1 598A8EB2
+P 1250 2250
+F 0 "10k?" V 1330 2250 50  0000 C CNN
+F 1 "R" V 1250 2250 50  0000 C CNN
+F 2 "" V 1180 2250 50  0001 C CNN
+F 3 "" H 1250 2250 50  0001 C CNN
+	1    1250 2250
+	0    -1   -1   0
+$EndComp
+$Comp
+L GND #PWR?
+U 1 1 598A8EB8
+P 950 2250
+F 0 "#PWR?" H 950 2000 50  0001 C CNN
+F 1 "GND" H 950 2100 50  0000 C CNN
+F 2 "" H 950 2250 50  0001 C CNN
+F 3 "" H 950 2250 50  0001 C CNN
+	1    950  2250
+	0    1    1    0
+$EndComp
+$Comp
+L SW_Push SW?
+U 1 1 598A8EBE
+P 1250 2050
+F 0 "SW?" H 1300 2150 50  0000 L CNN
+F 1 "SW_Push" H 1250 1990 50  0000 C CNN
+F 2 "" H 1250 2250 50  0001 C CNN
+F 3 "" H 1250 2250 50  0001 C CNN
+	1    1250 2050
+	1    0    0    -1
+$EndComp
+$Comp
+L +3.3V #PWR?
+U 1 1 598A8EC4
+P 950 2050
+F 0 "#PWR?" H 950 1900 50  0001 C CNN
+F 1 "+3.3V" H 950 2190 50  0000 C CNN
+F 2 "" H 950 2050 50  0001 C CNN
+F 3 "" H 950 2050 50  0001 C CNN
+	1    950  2050
+	0    -1   -1   0
+$EndComp
+Wire Wire Line
+	1100 2250 950  2250
+Wire Wire Line
+	1050 2050 950  2050
+Connection ~ 1450 2250
+Wire Wire Line
+	1450 2050 1450 2250
+Wire Wire Line
+	1400 2250 2550 2250
+Wire Wire Line
+	6050 5650 6050 5700
+Wire Wire Line
+	6050 5700 6450 5700
+Wire Wire Line
+	6450 5700 6450 5650
+Wire Wire Line
+	6350 5650 6350 5700
+Connection ~ 6350 5700
+Wire Wire Line
+	6250 5650 6250 5800
+Connection ~ 6250 5700
+Wire Wire Line
+	6150 5650 6150 5700
+Connection ~ 6150 5700
+$Comp
+L GND #PWR?
+U 1 1 598A971D
+P 6250 5800
+F 0 "#PWR?" H 6250 5550 50  0001 C CNN
+F 1 "GND" H 6250 5650 50  0000 C CNN
+F 2 "" H 6250 5800 50  0001 C CNN
+F 3 "" H 6250 5800 50  0001 C CNN
+	1    6250 5800
+	1    0    0    -1
+$EndComp
+Wire Wire Line
+	5400 1000 5400 1050
 Text HLabel 2550 3750 0    60   Input ~ 0
-BUS_TERM_CTRL
+prb_btn_1_pwr
+Text HLabel 2550 3850 0    60   Input ~ 0
+prb_btn_1_rs
+Text HLabel 2550 3950 0    60   Input ~ 0
+prb_LED_1_pwr
+Text HLabel 2550 4050 0    60   Input ~ 0
+prb_LED_1_rs
+Text HLabel 2550 4150 0    60   Input ~ 0
+prb_btn_2_pwr
+Text HLabel 2550 4250 0    60   Input ~ 0
+prb_btn_2_rs
+Text HLabel 2550 4350 0    60   Input ~ 0
+prb_LED_2_pwr
+Text HLabel 2550 4450 0    60   Input ~ 0
+prb_LED_2_rs
+Text HLabel 2550 4550 0    60   Input ~ 0
+prb_btn_3_pwr
+Text HLabel 2550 4650 0    60   Input ~ 0
+prb_btn_3_rs
+Text HLabel 2550 4750 0    60   Input ~ 0
+prb_LED_3_pwr
+Text HLabel 2550 4850 0    60   Input ~ 0
+prb_LED_3_rs
+Text HLabel 2550 4950 0    60   Input ~ 0
+prb_btn_4_pwr
+Text HLabel 2550 5050 0    60   Input ~ 0
+prb_btn_4_rs
+Text HLabel 2550 5150 0    60   Input ~ 0
+prb_LED_4_pwr
+Text HLabel 2550 5250 0    60   Input ~ 0
+prb_LED_4_rs
+Text HLabel 9950 2450 2    60   Input ~ 0
+prb_btn_pwr_master
+Text HLabel 9950 2550 2    60   Input ~ 0
+prb_btn_rs_master
 $EndSCHEMATC
