File: pt-module-mcu.sch (KiCad schematic (older format))
At the start: 14 parts

Commit message: Fixed missing components
Parts:
- C? (x2): renamed from 27pF; value C_Small -> 27pF
- R?: renamed from 10k; value R -> 10k
- R?: renamed from 10k?; value R -> 10k
Connections:
- net PRB_1_pwr_ctrl: now reaches U?.22 (ADC2_IN3/DAC2_OUT1/OPAMP2_DIG/OPAMP2_VOUT/SPI1_MISO/TIM16_CH1/TIM1_BKIN/TIM3_CH1/TSC_G2_IO3/PA6)
- net PRB_1_rs_ctrl: now reaches U?.23 (ADC2_IN4/COMP2_INP/OPAMP2_VINP/OPAMP2_VINP_SEC/SPI1_MOSI/TIM17_CH1/TIM1_CH1N/TIM3_CH2/TSC_G2_IO4/PA7)
- net PRB_3_pwr_ctrl: now reaches U?.26 (ADC1_IN11/COMP4_INP/OPAMP2_VINP/OPAMP2_VINP_SEC/TIM1_CH2N/TIM3_CH3/TSC_G3_IO2/PB0)
- net PRB_3_rs_ctrl: now reaches U?.27 (ADC1_IN12/COMP4_OUT/HRTIM1_SCOUT/TIM1_CH3N/TIM3_CH4/TSC_G3_IO3/PB1)
- net PRB_4_pwr_ctrl: now reaches U?.28 (ADC2_IN12/COMP4_INM/HRTIM1_SCIN/TSC_G3_IO4/PB2)
- net PRB_2_pwr_ctrl: now reaches U?.41 (HRTIM1_CHA1/RCC_MCO/TIM1_CH1/USART1_CK/PA8)
- net PRB_2_rs_ctrl: now reaches U?.42 (DAC1_EXTI9/DAC2_EXTI9/HRTIM1_CHA2/TIM15_BKIN/TIM1_CH2/TIM2_CH3/TSC_G4_IO1/USART1_TX/PA9)
- net PRB_4_rs_ctrl: now reaches U?.55 (HRTIM1_EEV9/HRTIM1_SCOUT/SPI1_SCK/SYS_JTDO-TRACESWO/TIM2_CH2/TIM3_ETR/TSC_G5_IO1/USART2_TX/PB3)
Changed lines of the file:
@@
 LIBS:ftdi
 LIBS:relays
-LIBS:components
 LIBS:pt-module-cache
 EELAYER 25 0
@@
 $EndComp
 $Comp
-L C_Small 27pF
+L C_Small C?
 U 1 1 597ECFD6
 P 1150 6600
-F 0 "27pF" H 1160 6670 50  0000 L CNN
-F 1 "C_Small" H 1160 6520 50  0000 L CNN
+F 0 "C?" H 1160 6670 50  0000 L CNN
+F 1 "27pF" H 1160 6520 50  0000 L CNN
 F 2 "" H 1150 6600 50  0001 C CNN
 F 3 "" H 1150 6600 50  0001 C CNN
@@
 $EndComp
 $Comp
-L C_Small 27pF
+L C_Small C?
 U 1 1 597ED20D
 P 1850 6600
-F 0 "27pF" H 1860 6670 50  0000 L CNN
-F 1 "C_Small" H 1860 6520 50  0000 L CNN
+F 0 "C?" H 1860 6670 50  0000 L CNN
+F 1 "27pF" H 1860 6520 50  0000 L CNN
 F 2 "" H 1850 6600 50  0001 C CNN
 F 3 "" H 1850 6600 50  0001 C CNN
@@
 RCC_OSC_IN
 $Comp
-L R 10k
+L R R?
 U 1 1 597EF7C5
 P 2050 2050
-F 0 "10k" V 2130 2050 50  0000 C CNN
-F 1 "R" V 2050 2050 50  0000 C CNN
+F 0 "R?" V 2130 2050 50  0000 C CNN
+F 1 "10k" V 2050 2050 50  0000 C CNN
 F 2 "" V 1980 2050 50  0001 C CNN
 F 3 "" H 2050 2050 50  0001 C CNN
@@
 BUS_TERM_CTRL
 $Comp
-L R 10k?
+L R R?
 U 1 1 598A8EB2
 P 1250 2250
-F 0 "10k?" V 1330 2250 50  0000 C CNN
-F 1 "R" V 1250 2250 50  0000 C CNN
+F 0 "R?" V 1330 2250 50  0000 C CNN
+F 1 "10k" V 1250 2250 50  0000 C CNN
 F 2 "" V 1180 2250 50  0001 C CNN
 F 3 "" H 1250 2250 50  0001 C CNN
@@
 Text HLabel 9950 2550 2    60   Input ~ 0
 prb_btn_rs_master
+Text HLabel 9950 2650 2    60   Input ~ 0
+PRB_1_pwr_ctrl
+Text HLabel 9950 2750 2    60   Input ~ 0
+PRB_1_rs_ctrl
+Text HLabel 9950 2950 2    60   Input ~ 0
+PRB_2_rs_ctrl
+Text HLabel 9950 2850 2    60   Input ~ 0
+PRB_2_pwr_ctrl
+Text HLabel 9950 3750 2    60   Input ~ 0
+PRB_3_pwr_ctrl
+Text HLabel 9950 3950 2    60   Input ~ 0
+PRB_4_pwr_ctrl
+Text HLabel 9950 3850 2    60   Input ~ 0
+PRB_3_rs_ctrl
+Text HLabel 9950 4050 2    60   Input ~ 0
+PRB_4_rs_ctrl
 $EndSCHEMATC

Commit message: Connected EVERYTHING. Ran ERC. There are still some power errors.
Parts:
- gave numbers to parts that had none: 13
- renumbered 16Mhz to 16Mhz1
Connections:
- no-connect marks 1 -> 13
Changed lines of the file:
@@
 LIBS:ftdi
 LIBS:relays
+LIBS:microchip_dspic33dsc
+LIBS:microchip_pic10mcu
+LIBS:microchip_pic12mcu
+LIBS:microchip_pic16mcu
+LIBS:microchip_pic18mcu
+LIBS:microchip_pic24mcu
+LIBS:microchip_pic32mcu
 LIBS:pt-module-cache
 EELAYER 25 0
@@
 $EndDescr
 $Comp
-L STM32F334R8Tx U?
+L STM32F334R8Tx U9
 U 1 1 597ECDC0
 P 6250 3650
-F 0 "U?" H 2650 5575 50  0000 L BNN
+F 0 "U9" H 2650 5575 50  0000 L BNN
 F 1 "STM32F334R8Tx" H 9850 5575 50  0000 R BNN
 F 2 "LQFP64" H 9850 5525 50  0001 R TNN
@@
 $EndComp
 $Comp
-L Crystal 16Mhz
+L Crystal 16Mhz1
 U 1 1 597ECED5
 P 1500 6400
-F 0 "16Mhz" H 1500 6550 50  0000 C CNN
+F 0 "16Mhz1" H 1500 6550 50  0000 C CNN
 F 1 "Crystal" H 1500 6250 50  0000 C CNN
 F 2 "" H 1500 6400 50  0001 C CNN
@@
 $EndComp
 $Comp
-L C_Small C?
+L C_Small C14
 U 1 1 597ECFD6
 P 1150 6600
-F 0 "C?" H 1160 6670 50  0000 L CNN
+F 0 "C14" H 1160 6670 50  0000 L CNN
 F 1 "27pF" H 1160 6520 50  0000 L CNN
 F 2 "" H 1150 6600 50  0001 C CNN
@@
 $EndComp
 $Comp
-L C_Small C?
+L C_Small C15
 U 1 1 597ED20D
 P 1850 6600
-F 0 "C?" H 1860 6670 50  0000 L CNN
+F 0 "C15" H 1860 6670 50  0000 L CNN
 F 1 "27pF" H 1860 6520 50  0000 L CNN
 F 2 "" H 1850 6600 50  0001 C CNN
@@
 $EndComp
 $Comp
-L GND #PWR031
+L GND #PWR079
 U 1 1 597EDE48
 P 1150 6800
-F 0 "#PWR031" H 1150 6550 50  0001 C CNN
+F 0 "#PWR079" H 1150 6550 50  0001 C CNN
 F 1 "GND" H 1150 6650 50  0000 C CNN
 F 2 "" H 1150 6800 50  0001 C CNN
@@
 $EndComp
 $Comp
-L GND #PWR032
+L GND #PWR080
 U 1 1 597EDE64
 P 1850 6800
-F 0 "#PWR032" H 1850 6550 50  0001 C CNN
+F 0 "#PWR080" H 1850 6550 50  0001 C CNN
 F 1 "GND" H 1850 6650 50  0000 C CNN
 F 2 "" H 1850 6800 50  0001 C CNN
@@
 RCC_OSC_IN
 $Comp
-L R R?
+L R R24
 U 1 1 597EF7C5
 P 2050 2050
-F 0 "R?" V 2130 2050 50  0000 C CNN
+F 0 "R24" V 2130 2050 50  0000 C CNN
 F 1 "10k" V 2050 2050 50  0000 C CNN
 F 2 "" V 1980 2050 50  0001 C CNN
@@
 $EndComp
 $Comp
-L GND #PWR033
+L GND #PWR081
 U 1 1 597EF838
 P 1750 1850
-F 0 "#PWR033" H 1750 1600 50  0001 C CNN
+F 0 "#PWR081" H 1750 1600 50  0001 C CNN
 F 1 "GND" H 1750 1700 50  0000 C CNN
 F 2 "" H 1750 1850 50  0001 C CNN
@@
 $EndComp
 $Comp
-L SW_Push SW?
+L SW_Push SW9
 U 1 1 597EF85E
 P 2050 1850
-F 0 "SW?" H 2100 1950 50  0000 L CNN
+F 0 "SW9" H 2100 1950 50  0000 L CNN
 F 1 "SW_Push" H 2050 1790 50  0000 C CNN
 F 2 "" H 2050 2050 50  0001 C CNN
@@
 $EndComp
 $Comp
-L C_Small C?
+L C_Small C17
 U 1 1 597F1898
 P 6000 1100
-F 0 "C?" H 6010 1170 50  0000 L CNN
+F 0 "C17" H 6010 1170 50  0000 L CNN
 F 1 "C_Small" H 6010 1020 50  0000 L CNN
 F 2 "" H 6000 1100 50  0001 C CNN
@@
 $EndComp
 $Comp
-L C_Small C?
+L C_Small C18
 U 1 1 597F1903
 P 6200 1100
-F 0 "C?" H 6210 1170 50  0000 L CNN
+F 0 "C18" H 6210 1170 50  0000 L CNN
 F 1 "C_Small" H 6210 1020 50  0000 L CNN
 F 2 "" H 6200 1100 50  0001 C CNN
@@
 $EndComp
 $Comp
-L C_Small C?
+L C_Small C19
 U 1 1 597F1997
 P 6400 1100
-F 0 "C?" H 6410 1170 50  0000 L CNN
+F 0 "C19" H 6410 1170 50  0000 L CNN
 F 1 "C_Small" H 6410 1020 50  0000 L CNN
 F 2 "" H 6400 1100 50  0001 C CNN
@@
 $EndComp
 $Comp
-L C_Small C?
+L C_Small C20
 U 1 1 597F19E6
 P 6600 1100
-F 0 "C?" H 6610 1170 50  0000 L CNN
+F 0 "C20" H 6610 1170 50  0000 L CNN
 F 1 "C_Small" H 6610 1020 50  0000 L CNN
 F 2 "" H 6600 1100 50  0001 C CNN
@@
 $EndComp
 $Comp
-L C_Small C?
+L C_Small C16
 U 1 1 597F1A58
 P 5800 1100
-F 0 "C?" H 5810 1170 50  0000 L CNN
+F 0 "C16" H 5810 1170 50  0000 L CNN
 F 1 "C_Small" H 5810 1020 50  0000 L CNN
 F 2 "" H 5800 1100 50  0001 C CNN
@@
 $EndComp
 $Comp
-L C_Small C?
+L C_Small C21
 U 1 1 597F1AA1
 P 6800 1100
-F 0 "C?" H 6810 1170 50  0000 L CNN
+F 0 "C21" H 6810 1170 50  0000 L CNN
 F 1 "C_Small" H 6810 1020 50  0000 L CNN
 F 2 "" H 6800 1100 50  0001 C CNN
@@
 $EndComp
 $Comp
-L GND #PWR034
+L GND #PWR082
 U 1 1 597F238E
 P 5400 1050
-F 0 "#PWR034" H 5400 800 50  0001 C CNN
+F 0 "#PWR082" H 5400 800 50  0001 C CNN
 F 1 "GND" H 5400 900 50  0000 C CNN
 F 2 "" H 5400 1050 50  0001 C CNN
@@
 NoConn ~ 2550 2450
 $Comp
-L +3.3V #PWR035
+L +3.3V #PWR083
 U 1 1 5980C7A4
 P 5900 1650
-F 0 "#PWR035" H 5900 1500 50  0001 C CNN
+F 0 "#PWR083" H 5900 1500 50  0001 C CNN
 F 1 "+3.3V" H 5900 1790 50  0000 C CNN
 F 2 "" H 5900 1650 50  0001 C CNN
@@
 $EndComp
 $Comp
-L +3.3V #PWR036
+L +3.3V #PWR084
 U 1 1 5980CC21
 P 1750 2050
-F 0 "#PWR036" H 1750 1900 50  0001 C CNN
+F 0 "#PWR084" H 1750 1900 50  0001 C CNN
 F 1 "+3.3V" H 1750 2190 50  0000 C CNN
 F 2 "" H 1750 2050 50  0001 C CNN
@@
 BUS_TERM_CTRL
 $Comp
-L R R?
+L R R23
 U 1 1 598A8EB2
 P 1250 2250
-F 0 "R?" V 1330 2250 50  0000 C CNN
+F 0 "R23" V 1330 2250 50  0000 C CNN
 F 1 "10k" V 1250 2250 50  0000 C CNN
 F 2 "" V 1180 2250 50  0001 C CNN
@@
 $EndComp
 $Comp
-L GND #PWR?
+L GND #PWR085
 U 1 1 598A8EB8
 P 950 2250
-F 0 "#PWR?" H 950 2000 50  0001 C CNN
+F 0 "#PWR085" H 950 2000 50  0001 C CNN
 F 1 "GND" H 950 2100 50  0000 C CNN
 F 2 "" H 950 2250 50  0001 C CNN
@@
 $EndComp
 $Comp
-L SW_Push SW?
+L SW_Push SW8
 U 1 1 598A8EBE
 P 1250 2050
-F 0 "SW?" H 1300 2150 50  0000 L CNN
+F 0 "SW8" H 1300 2150 50  0000 L CNN
 F 1 "SW_Push" H 1250 1990 50  0000 C CNN
 F 2 "" H 1250 2250 50  0001 C CNN
@@
 $EndComp
 $Comp
-L +3.3V #PWR?
+L +3.3V #PWR086
 U 1 1 598A8EC4
 P 950 2050
-F 0 "#PWR?" H 950 1900 50  0001 C CNN
+F 0 "#PWR086" H 950 1900 50  0001 C CNN
 F 1 "+3.3V" H 950 2190 50  0000 C CNN
 F 2 "" H 950 2050 50  0001 C CNN
@@
 Connection ~ 6150 5700
 $Comp
-L GND #PWR?
+L GND #PWR087
 U 1 1 598A971D
 P 6250 5800
-F 0 "#PWR?" H 6250 5550 50  0001 C CNN
+F 0 "#PWR087" H 6250 5550 50  0001 C CNN
 F 1 "GND" H 6250 5650 50  0000 C CNN
 F 2 "" H 6250 5800 50  0001 C CNN
@@
 Text HLabel 9950 4050 2    60   Input ~ 0
 PRB_4_rs_ctrl
+NoConn ~ 2550 3550
+NoConn ~ 9950 3050
+NoConn ~ 9950 3350
+NoConn ~ 9950 3450
+NoConn ~ 9950 3550
+NoConn ~ 9950 2050
+NoConn ~ 9950 4150
+NoConn ~ 9950 4250
+NoConn ~ 9950 4750
+NoConn ~ 9950 4850
+NoConn ~ 9950 4950
+NoConn ~ 9950 5050
 $EndSCHEMATC

Commit message: Re-annotation
Parts:
- renumbered R23 to R25, R24 to R26, U9 to U8
Changed lines of the file:
@@
 $EndDescr
 $Comp
-L STM32F334R8Tx U9
+L STM32F334R8Tx U8
 U 1 1 597ECDC0
 P 6250 3650
-F 0 "U9" H 2650 5575 50  0000 L BNN
+F 0 "U8" H 2650 5575 50  0000 L BNN
 F 1 "STM32F334R8Tx" H 9850 5575 50  0000 R BNN
 F 2 "LQFP64" H 9850 5525 50  0001 R TNN
@@
 $EndComp
 $Comp
-L GND #PWR079
+L GND #PWR74
 U 1 1 597EDE48
 P 1150 6800
-F 0 "#PWR079" H 1150 6550 50  0001 C CNN
+F 0 "#PWR74" H 1150 6550 50  0001 C CNN
 F 1 "GND" H 1150 6650 50  0000 C CNN
 F 2 "" H 1150 6800 50  0001 C CNN
@@
 $EndComp
 $Comp
-L GND #PWR080
+L GND #PWR77
 U 1 1 597EDE64
 P 1850 6800
-F 0 "#PWR080" H 1850 6550 50  0001 C CNN
+F 0 "#PWR77" H 1850 6550 50  0001 C CNN
 F 1 "GND" H 1850 6650 50  0000 C CNN
 F 2 "" H 1850 6800 50  0001 C CNN
@@
 RCC_OSC_IN
 $Comp
-L R R24
+L R R26
 U 1 1 597EF7C5
 P 2050 2050
-F 0 "R24" V 2130 2050 50  0000 C CNN
+F 0 "R26" V 2130 2050 50  0000 C CNN
 F 1 "10k" V 2050 2050 50  0000 C CNN
 F 2 "" V 1980 2050 50  0001 C CNN
@@
 $EndComp
 $Comp
-L GND #PWR081
+L GND #PWR75
 U 1 1 597EF838
 P 1750 1850
-F 0 "#PWR081" H 1750 1600 50  0001 C CNN
+F 0 "#PWR75" H 1750 1600 50  0001 C CNN
 F 1 "GND" H 1750 1700 50  0000 C CNN
 F 2 "" H 1750 1850 50  0001 C CNN
@@
 $EndComp
 $Comp
-L GND #PWR082
+L GND #PWR78
 U 1 1 597F238E
 P 5400 1050
-F 0 "#PWR082" H 5400 800 50  0001 C CNN
+F 0 "#PWR78" H 5400 800 50  0001 C CNN
 F 1 "GND" H 5400 900 50  0000 C CNN
 F 2 "" H 5400 1050 50  0001 C CNN
@@
 NoConn ~ 2550 2450
 $Comp
-L +3.3V #PWR083
+L +3.3V #PWR79
 U 1 1 5980C7A4
 P 5900 1650
-F 0 "#PWR083" H 5900 1500 50  0001 C CNN
+F 0 "#PWR79" H 5900 1500 50  0001 C CNN
 F 1 "+3.3V" H 5900 1790 50  0000 C CNN
 F 2 "" H 5900 1650 50  0001 C CNN
@@
 $EndComp
 $Comp
-L +3.3V #PWR084
+L +3.3V #PWR76
 U 1 1 5980CC21
 P 1750 2050
-F 0 "#PWR084" H 1750 1900 50  0001 C CNN
+F 0 "#PWR76" H 1750 1900 50  0001 C CNN
 F 1 "+3.3V" H 1750 2190 50  0000 C CNN
 F 2 "" H 1750 2050 50  0001 C CNN
@@
 BUS_TERM_CTRL
 $Comp
-L R R23
+L R R25
 U 1 1 598A8EB2
 P 1250 2250
-F 0 "R23" V 1330 2250 50  0000 C CNN
+F 0 "R25" V 1330 2250 50  0000 C CNN
 F 1 "10k" V 1250 2250 50  0000 C CNN
 F 2 "" V 1180 2250 50  0001 C CNN
@@
 $EndComp
 $Comp
-L GND #PWR085
+L GND #PWR73
 U 1 1 598A8EB8
 P 950 2250
-F 0 "#PWR085" H 950 2000 50  0001 C CNN
+F 0 "#PWR73" H 950 2000 50  0001 C CNN
 F 1 "GND" H 950 2100 50  0000 C CNN
 F 2 "" H 950 2250 50  0001 C CNN
@@
 $EndComp
 $Comp
-L +3.3V #PWR086
+L +3.3V #PWR72
 U 1 1 598A8EC4
 P 950 2050
-F 0 "#PWR086" H 950 1900 50  0001 C CNN
+F 0 "#PWR72" H 950 1900 50  0001 C CNN
 F 1 "+3.3V" H 950 2190 50  0000 C CNN
 F 2 "" H 950 2050 50  0001 C CNN
@@
 Connection ~ 6150 5700
 $Comp
-L GND #PWR087
+L GND #PWR80
 U 1 1 598A971D
 P 6250 5800
-F 0 "#PWR087" H 6250 5550 50  0001 C CNN
+F 0 "#PWR80" H 6250 5550 50  0001 C CNN
 F 1 "GND" H 6250 5650 50  0000 C CNN
 F 2 "" H 6250 5800 50  0001 C CNN
