File: pt-module-interface-master.sch (KiCad schematic (older format))
At the start: 4 parts

Commit message: Connected EVERYTHING. Ran ERC. There are still some power errors.
Parts:
- R25, R26: renamed from R?; value R -> 10k
- gave numbers to parts that had none: 2
Changed lines of the file:
@@
 LIBS:ftdi
 LIBS:relays
+LIBS:microchip_dspic33dsc
+LIBS:microchip_pic10mcu
+LIBS:microchip_pic12mcu
+LIBS:microchip_pic16mcu
+LIBS:microchip_pic18mcu
+LIBS:microchip_pic24mcu
+LIBS:microchip_pic32mcu
 LIBS:pt-module-cache
 EELAYER 25 0
@@
 $EndDescr
 $Comp
-L SW_Push SW?
+L SW_Push SW10
 U 1 1 598EE80D
 P 4350 2350
-F 0 "SW?" H 4400 2450 50  0000 L CNN
+F 0 "SW10" H 4400 2450 50  0000 L CNN
 F 1 "SW_Push" H 4350 2290 50  0000 C CNN
 F 2 "" H 4350 2550 50  0001 C CNN
@@
 $EndComp
 $Comp
-L GND #PWR?
+L GND #PWR088
 U 1 1 598EE82A
 P 4000 2400
-F 0 "#PWR?" H 4000 2150 50  0001 C CNN
+F 0 "#PWR088" H 4000 2150 50  0001 C CNN
 F 1 "GND" H 4000 2250 50  0000 C CNN
 F 2 "" H 4000 2400 50  0001 C CNN
@@
 $EndComp
 $Comp
-L +3.3V #PWR?
+L +3.3V #PWR089
 U 1 1 598EE89F
 P 4700 1900
-F 0 "#PWR?" H 4700 1750 50  0001 C CNN
+F 0 "#PWR089" H 4700 1750 50  0001 C CNN
 F 1 "+3.3V" H 4700 2040 50  0000 C CNN
 F 2 "" H 4700 1900 50  0001 C CNN
@@
 	4000 2350 4000 2400
 $Comp
-L R R?
+L R R25
 U 1 1 598F39A9
 P 4700 2150
-F 0 "R?" V 4780 2150 50  0000 C CNN
-F 1 "R" V 4700 2150 50  0000 C CNN
+F 0 "R25" V 4780 2150 50  0000 C CNN
+F 1 "10k" V 4700 2150 50  0000 C CNN
 F 2 "" V 4630 2150 50  0001 C CNN
 F 3 "" H 4700 2150 50  0001 C CNN
@@
 Connection ~ 4700 2350
 $Comp
-L SW_Push SW?
+L SW_Push SW11
 U 1 1 598F3B30
 P 4350 3250
-F 0 "SW?" H 4400 3350 50  0000 L CNN
+F 0 "SW11" H 4400 3350 50  0000 L CNN
 F 1 "SW_Push" H 4350 3190 50  0000 C CNN
 F 2 "" H 4350 3450 50  0001 C CNN
@@
 $EndComp
 $Comp
-L GND #PWR?
+L GND #PWR090
 U 1 1 598F3B36
 P 4000 3300
-F 0 "#PWR?" H 4000 3050 50  0001 C CNN
+F 0 "#PWR090" H 4000 3050 50  0001 C CNN
 F 1 "GND" H 4000 3150 50  0000 C CNN
 F 2 "" H 4000 3300 50  0001 C CNN
@@
 $EndComp
 $Comp
-L +3.3V #PWR?
+L +3.3V #PWR091
 U 1 1 598F3B3C
 P 4700 2800
-F 0 "#PWR?" H 4700 2650 50  0001 C CNN
+F 0 "#PWR091" H 4700 2650 50  0001 C CNN
 F 1 "+3.3V" H 4700 2940 50  0000 C CNN
 F 2 "" H 4700 2800 50  0001 C CNN
@@
 	4000 3250 4000 3300
 $Comp
-L R R?
+L R R26
 U 1 1 598F3B45
 P 4700 3050
-F 0 "R?" V 4780 3050 50  0000 C CNN
-F 1 "R" V 4700 3050 50  0000 C CNN
+F 0 "R26" V 4780 3050 50  0000 C CNN
+F 1 "10k" V 4700 3050 50  0000 C CNN
 F 2 "" V 4630 3050 50  0001 C CNN
 F 3 "" H 4700 3050 50  0001 C CNN

Commit message: Re-annotation
Parts:
- renumbered R25 to R27, R26 to R28
Changed lines of the file:
@@
 $EndComp
 $Comp
-L GND #PWR088
+L GND #PWR81
 U 1 1 598EE82A
 P 4000 2400
-F 0 "#PWR088" H 4000 2150 50  0001 C CNN
+F 0 "#PWR81" H 4000 2150 50  0001 C CNN
 F 1 "GND" H 4000 2250 50  0000 C CNN
 F 2 "" H 4000 2400 50  0001 C CNN
@@
 $EndComp
 $Comp
-L +3.3V #PWR089
+L +3.3V #PWR83
 U 1 1 598EE89F
 P 4700 1900
-F 0 "#PWR089" H 4700 1750 50  0001 C CNN
+F 0 "#PWR83" H 4700 1750 50  0001 C CNN
 F 1 "+3.3V" H 4700 2040 50  0000 C CNN
 F 2 "" H 4700 1900 50  0001 C CNN
@@
 	4000 2350 4000 2400
 $Comp
-L R R25
+L R R27
 U 1 1 598F39A9
 P 4700 2150
-F 0 "R25" V 4780 2150 50  0000 C CNN
+F 0 "R27" V 4780 2150 50  0000 C CNN
 F 1 "10k" V 4700 2150 50  0000 C CNN
 F 2 "" V 4630 2150 50  0001 C CNN
@@
 $EndComp
 $Comp
-L GND #PWR090
+L GND #PWR82
 U 1 1 598F3B36
 P 4000 3300
-F 0 "#PWR090" H 4000 3050 50  0001 C CNN
+F 0 "#PWR82" H 4000 3050 50  0001 C CNN
 F 1 "GND" H 4000 3150 50  0000 C CNN
 F 2 "" H 4000 3300 50  0001 C CNN
@@
 $EndComp
 $Comp
-L +3.3V #PWR091
+L +3.3V #PWR84
 U 1 1 598F3B3C
 P 4700 2800
-F 0 "#PWR091" H 4700 2650 50  0001 C CNN
+F 0 "#PWR84" H 4700 2650 50  0001 C CNN
 F 1 "+3.3V" H 4700 2940 50  0000 C CNN
 F 2 "" H 4700 2800 50  0001 C CNN
@@
 	4000 3250 4000 3300
 $Comp
-L R R26
+L R R28
 U 1 1 598F3B45
 P 4700 3050
-F 0 "R26" V 4780 3050 50  0000 C CNN
+F 0 "R28" V 4780 3050 50  0000 C CNN
 F 1 "10k" V 4700 3050 50  0000 C CNN
 F 2 "" V 4630 3050 50  0001 C CNN
