File: pt-module-interface-master.sch (KiCad schematic (older format))
At the start: 4 parts, among them SW10 SW_Push, SW11 SW_Push

Commit message: add all the rest of the footprints
Parts:
- R27, R28: footprint (none) -> Resistors_SMD:R_1206_HandSoldering
- SW10, SW11: footprint (none) -> Connectors_Hirose:Hirose_DF13C-02P-1.25V_02x1.25mm_Straight
Changed lines of the file:
@@
 F 0 "SW10" H 4400 2450 50  0000 L CNN
 F 1 "SW_Push" H 4350 2290 50  0000 C CNN
-F 2 "" H 4350 2550 50  0001 C CNN
+F 2 "Connectors_Hirose:Hirose_DF13C-02P-1.25V_02x1.25mm_Straight" H 4350 2550 50  0001 C CNN
 F 3 "" H 4350 2550 50  0001 C CNN
 	1    4350 2350
@@
 F 0 "R27" V 4780 2150 50  0000 C CNN
 F 1 "10k" V 4700 2150 50  0000 C CNN
-F 2 "" V 4630 2150 50  0001 C CNN
+F 2 "Resistors_SMD:R_1206_HandSoldering" V 4630 2150 50  0001 C CNN
 F 3 "" H 4700 2150 50  0001 C CNN
 	1    4700 2150
@@
 F 0 "SW11" H 4400 3350 50  0000 L CNN
 F 1 "SW_Push" H 4350 3190 50  0000 C CNN
-F 2 "" H 4350 3450 50  0001 C CNN
+F 2 "Connectors_Hirose:Hirose_DF13C-02P-1.25V_02x1.25mm_Straight" H 4350 3450 50  0001 C CNN
 F 3 "" H 4350 3450 50  0001 C CNN
 	1    4350 3250
@@
 F 0 "R28" V 4780 3050 50  0000 C CNN
 F 1 "10k" V 4700 3050 50  0000 C CNN
-F 2 "" V 4630 3050 50  0001 C CNN
+F 2 "Resistors_SMD:R_1206_HandSoldering" V 4630 3050 50  0001 C CNN
 F 3 "" H 4700 3050 50  0001 C CNN
 	1    4700 3050
