File: pt-module-rs485.sch (KiCad schematic (older format))
At the start: 10 parts, among them U3 SN65HVD72, U4 SN65HVD72

Commit message: add all the rest of the footprints
Parts:
- C10, C9: footprint (none) -> Capacitors_SMD:C_1206_HandSoldering
- D6, D7: footprint (none) -> Diodes_SMD:D_SOT-23_ANK
- R5, R6, R7, R8: footprint (none) -> Resistors_SMD:R_0805_HandSoldering
Changed lines of the file:
@@
 F 0 "R7" V 6080 5000 50  0000 C CNN
 F 1 "10R" V 6000 5000 50  0000 C CNN
-F 2 "" V 5930 5000 50  0001 C CNN
+F 2 "Resistors_SMD:R_0805_HandSoldering" V 5930 5000 50  0001 C CNN
 F 3 "" H 6000 5000 50  0001 C CNN
 	1    6000 5000
@@
 F 0 "R8" V 6080 5200 50  0000 C CNN
 F 1 "10R" V 6000 5200 50  0000 C CNN
-F 2 "" V 5930 5200 50  0001 C CNN
+F 2 "Resistors_SMD:R_0805_HandSoldering" V 5930 5200 50  0001 C CNN
 F 3 "" H 6000 5200 50  0001 C CNN
 	1    6000 5200
@@
 F 0 "C10" H 5810 4770 50  0000 L CNN
 F 1 "100nF" H 5810 4620 50  0000 L CNN
-F 2 "" H 5800 4700 50  0001 C CNN
+F 2 "Capacitors_SMD:C_1206_HandSoldering" H 5800 4700 50  0001 C CNN
 F 3 "" H 5800 4700 50  0001 C CNN
 	1    5800 4700
@@
 F 0 "D7" H 6500 5275 50  0000 C CNN
 F 1 "SM712" H 6500 5200 50  0000 C CNN
-F 2 "" H 6350 5100 50  0001 C CNN
+F 2 "Diodes_SMD:D_SOT-23_ANK" H 6350 5100 50  0001 C CNN
 F 3 "" H 6350 5100 50  0001 C CNN
 	1    6500 5100
@@
 F 0 "C9" H 5810 2120 50  0000 L CNN
 F 1 "100nF" H 5810 1970 50  0000 L CNN
-F 2 "" H 5800 2050 50  0001 C CNN
+F 2 "Capacitors_SMD:C_1206_HandSoldering" H 5800 2050 50  0001 C CNN
 F 3 "" H 5800 2050 50  0001 C CNN
 	1    5800 2050
@@
 F 0 "R5" V 6080 2350 50  0000 C CNN
 F 1 "10R" V 6000 2350 50  0000 C CNN
-F 2 "" V 5930 2350 50  0001 C CNN
+F 2 "Resistors_SMD:R_0805_HandSoldering" V 5930 2350 50  0001 C CNN
 F 3 "" H 6000 2350 50  0001 C CNN
 	1    6000 2350
@@
 F 0 "R6" V 6080 2550 50  0000 C CNN
 F 1 "10R" V 6000 2550 50  0000 C CNN
-F 2 "" V 5930 2550 50  0001 C CNN
+F 2 "Resistors_SMD:R_0805_HandSoldering" V 5930 2550 50  0001 C CNN
 F 3 "" H 6000 2550 50  0001 C CNN
 	1    6000 2550
@@
 F 0 "D6" H 6500 2625 50  0000 C CNN
 F 1 "SM712" H 6500 2550 50  0000 C CNN
-F 2 "" H 6350 2450 50  0001 C CNN
+F 2 "Diodes_SMD:D_SOT-23_ANK" H 6350 2450 50  0001 C CNN
 F 3 "" H 6350 2450 50  0001 C CNN
 	1    6500 2450

Commit message: fix footprint errors
Parts:
- D6, D7: footprint Diodes_SMD:D_SOT-23_ANK -> TO_SOT_Packages_SMD:SOT-23_Handsoldering
Changed lines of the file:
@@
 F 0 "D7" H 6500 5275 50  0000 C CNN
 F 1 "SM712" H 6500 5200 50  0000 C CNN
-F 2 "Diodes_SMD:D_SOT-23_ANK" H 6350 5100 50  0001 C CNN
+F 2 "TO_SOT_Packages_SMD:SOT-23_Handsoldering" H 6350 5100 50  0001 C CNN
 F 3 "" H 6350 5100 50  0001 C CNN
 	1    6500 5100
@@
 F 0 "D6" H 6500 2625 50  0000 C CNN
 F 1 "SM712" H 6500 2550 50  0000 C CNN
-F 2 "Diodes_SMD:D_SOT-23_ANK" H 6350 2450 50  0001 C CNN
+F 2 "TO_SOT_Packages_SMD:SOT-23_Handsoldering" H 6350 2450 50  0001 C CNN
 F 3 "" H 6350 2450 50  0001 C CNN
 	1    6500 2450
