File: probe_module2.sch (KiCad schematic (older format))
At the start: 4 parts, among them J6 CONN_01X05, J7 CONN_01X05, U6 DG411, U7 LH1526

Commit message: Connected EVERYTHING. Ran ERC. There are still some power errors.
Connections:
- net prb1_pwr_ctrl renamed prb3_pwr_ctrl
- net prb1_rs_ctrl renamed prb3_rs_ctrl
- net prb2_pwr_ctrl renamed prb4_pwr_ctrl
- net prb2_rs_ctrl renamed prb4_rs_ctrl
Changed lines of the file:
@@
 $Descr A4 11693 8268
 encoding utf-8
-Sheet 4 13
+Sheet 13 13
 Title ""
 Date ""
@@
 AR Path="/598183C5/5981A21D" Ref="U6"  Part="1"
 AR Path="/59933B07/5981A21D" Ref="U10"  Part="1"
-F 0 "U6" H 2300 4550 50  0000 C CNN
+F 0 "U10" H 2300 4550 50  0000 C CNN
 F 1 "DG411" H 2300 4350 50  0000 C CNN
 F 2 "" H 2300 4450 60  0001 C CNN
@@
 P 2350 4950
 AR Path="/598183C5/5981A4AC" Ref="#PWR041"  Part="1"
-AR Path="/59933B07/5981A4AC" Ref="#PWR95"  Part="1"
-F 0 "#PWR041" H 2350 4700 50  0001 C CNN
+AR Path="/59933B07/5981A4AC" Ref="#PWR098"  Part="1"
+F 0 "#PWR098" H 2350 4700 50  0001 C CNN
 F 1 "GND" H 2350 4800 50  0000 C CNN
 F 2 "" H 2350 4950 50  0001 C CNN
@@
 P 4700 4950
 AR Path="/598183C5/5981A5BD" Ref="#PWR042"  Part="1"
-AR Path="/59933B07/5981A5BD" Ref="#PWR98"  Part="1"
-F 0 "#PWR042" H 4700 4700 50  0001 C CNN
+AR Path="/59933B07/5981A5BD" Ref="#PWR099"  Part="1"
+F 0 "#PWR099" H 4700 4700 50  0001 C CNN
 F 1 "GND" H 4700 4800 50  0000 C CNN
 F 2 "" H 4700 4950 50  0001 C CNN
@@
 P 2350 3950
 AR Path="/598183C5/5981A680" Ref="#PWR043"  Part="1"
-AR Path="/59933B07/5981A680" Ref="#PWR94"  Part="1"
-F 0 "#PWR043" H 2350 3800 50  0001 C CNN
+AR Path="/59933B07/5981A680" Ref="#PWR0100"  Part="1"
+F 0 "#PWR0100" H 2350 3800 50  0001 C CNN
 F 1 "+3.3V" H 2350 4090 50  0000 C CNN
 F 2 "" H 2350 3950 50  0001 C CNN
@@
 P 4700 3950
 AR Path="/598183C5/5981A69E" Ref="#PWR044"  Part="1"
-AR Path="/59933B07/5981A69E" Ref="#PWR97"  Part="1"
-F 0 "#PWR044" H 4700 3800 50  0001 C CNN
+AR Path="/59933B07/5981A69E" Ref="#PWR0101"  Part="1"
+F 0 "#PWR0101" H 4700 3800 50  0001 C CNN
 F 1 "+3.3V" H 4700 4090 50  0000 C CNN
 F 2 "" H 4700 3950 50  0001 C CNN
@@
 AR Path="/598183C5/5981A26A" Ref="U6"  Part="2"
 AR Path="/59933B07/5981A26A" Ref="U10"  Part="2"
-F 0 "U6" H 4650 4550 50  0000 C CNN
+F 0 "U10" H 4650 4550 50  0000 C CNN
 F 1 "DG411" H 4650 4350 50  0000 C CNN
 F 2 "" H 4650 4450 60  0001 C CNN
@@
 prb1_b
 Text HLabel 5250 3000 3    60   Input ~ 0
-prb1_pwr_ctrl
+prb3_pwr_ctrl
 Text HLabel 1850 4350 0    60   Input ~ 0
-prb1_rs_ctrl
+prb3_rs_ctrl
 Text HLabel 1850 4550 0    60   Input ~ 0
 vaisala_rs485_a
 Text HLabel 4200 4350 0    60   Input ~ 0
-prb1_rs_ctrl
+prb3_rs_ctrl
 Text HLabel 5100 4550 2    60   Input ~ 0
 vaisala_rs485_b
@@
 AR Path="/598183C5/5981EAC3" Ref="U6"  Part="3"
 AR Path="/59933B07/5981EAC3" Ref="U10"  Part="3"
-F 0 "U6" H 7400 4550 50  0000 C CNN
+F 0 "U10" H 7400 4550 50  0000 C CNN
 F 1 "DG411" H 7400 4350 50  0000 C CNN
 F 2 "" H 7400 4450 60  0001 C CNN
@@
 P 7450 4950
 AR Path="/598183C5/5981EAC9" Ref="#PWR045"  Part="1"
-AR Path="/59933B07/5981EAC9" Ref="#PWR104"  Part="1"
-F 0 "#PWR045" H 7450 4700 50  0001 C CNN
+AR Path="/59933B07/5981EAC9" Ref="#PWR0102"  Part="1"
+F 0 "#PWR0102" H 7450 4700 50  0001 C CNN
 F 1 "GND" H 7450 4800 50  0000 C CNN
 F 2 "" H 7450 4950 50  0001 C CNN
@@
 P 9500 4900
 AR Path="/598183C5/5981EACF" Ref="#PWR046"  Part="1"
-AR Path="/59933B07/5981EACF" Ref="#PWR107"  Part="1"
-F 0 "#PWR046" H 9500 4650 50  0001 C CNN
+AR Path="/59933B07/5981EACF" Ref="#PWR0103"  Part="1"
+F 0 "#PWR0103" H 9500 4650 50  0001 C CNN
 F 1 "GND" H 9500 4750 50  0000 C CNN
 F 2 "" H 9500 4900 50  0001 C CNN
@@
 P 7450 3950
 AR Path="/598183C5/5981EAD5" Ref="#PWR047"  Part="1"
-AR Path="/59933B07/5981EAD5" Ref="#PWR103"  Part="1"
-F 0 "#PWR047" H 7450 3800 50  0001 C CNN
+AR Path="/59933B07/5981EAD5" Ref="#PWR0104"  Part="1"
+F 0 "#PWR0104" H 7450 3800 50  0001 C CNN
 F 1 "+3.3V" H 7450 4090 50  0000 C CNN
 F 2 "" H 7450 3950 50  0001 C CNN
@@
 P 9500 3900
 AR Path="/598183C5/5981EADB" Ref="#PWR048"  Part="1"
-AR Path="/59933B07/5981EADB" Ref="#PWR106"  Part="1"
-F 0 "#PWR048" H 9500 3750 50  0001 C CNN
+AR Path="/59933B07/5981EADB" Ref="#PWR0105"  Part="1"
+F 0 "#PWR0105" H 9500 3750 50  0001 C CNN
 F 1 "+3.3V" H 9500 4040 50  0000 C CNN
 F 2 "" H 9500 3900 50  0001 C CNN
@@
 AR Path="/598183C5/5981EAE3" Ref="U6"  Part="4"
 AR Path="/59933B07/5981EAE3" Ref="U10"  Part="4"
-F 0 "U6" H 9450 4500 50  0000 C CNN
+F 0 "U10" H 9450 4500 50  0000 C CNN
 F 1 "DG411" H 9450 4300 50  0000 C CNN
 F 2 "" H 9450 4400 60  0001 C CNN
@@
 $EndComp
 Text HLabel 6950 4350 0    60   Input ~ 0
-prb2_rs_ctrl
+prb4_rs_ctrl
 Text HLabel 6950 4550 0    60   Input ~ 0
 vaisala_rs485_a
 Text HLabel 9000 4300 0    60   Input ~ 0
-prb2_rs_ctrl
+prb4_rs_ctrl
 Text HLabel 9900 4500 2    60   Input ~ 0
 vaisala_rs485_b
@@
 AR Path="/598183C5/598215F3" Ref="J6"  Part="1"
 AR Path="/59933B07/598215F3" Ref="J9"  Part="1"
-F 0 "J6" H 3100 2000 50  0000 C CNN
+F 0 "J9" H 3100 2000 50  0000 C CNN
 F 1 "CONN_01X05" V 3200 1700 50  0000 C CNN
 F 2 "" H 3100 1700 50  0001 C CNN
@@
 NoConn ~ 3300 1900
 Text HLabel 5450 3000 3    60   Input ~ 0
-prb2_pwr_ctrl
+prb4_pwr_ctrl
 $Comp
 L CONN_01X05 J7
@@
 AR Path="/598183C5/59821868" Ref="J7"  Part="1"
 AR Path="/59933B07/59821868" Ref="J10"  Part="1"
-F 0 "J7" H 8000 1900 50  0000 C CNN
+F 0 "J10" H 8000 1900 50  0000 C CNN
 F 1 "CONN_01X05" V 8100 1600 50  0000 C CNN
 F 2 "" H 8000 1600 50  0001 C CNN
@@
 P 5350 2750
 AR Path="/598183C5/5990A260" Ref="#PWR049"  Part="1"
-AR Path="/59933B07/5990A260" Ref="#PWR100"  Part="1"
-F 0 "#PWR049" H 5350 2500 50  0001 C CNN
+AR Path="/59933B07/5990A260" Ref="#PWR0106"  Part="1"
+F 0 "#PWR0106" H 5350 2500 50  0001 C CNN
 F 1 "GND" H 5350 2600 50  0000 C CNN
 F 2 "" H 5350 2750 50  0001 C CNN
@@
 P 5550 2750
 AR Path="/598183C5/5990A28D" Ref="#PWR050"  Part="1"
-AR Path="/59933B07/5990A28D" Ref="#PWR102"  Part="1"
-F 0 "#PWR050" H 5550 2500 50  0001 C CNN
+AR Path="/59933B07/5990A28D" Ref="#PWR0107"  Part="1"
+F 0 "#PWR0107" H 5550 2500 50  0001 C CNN
 F 1 "GND" H 5550 2600 50  0000 C CNN
 F 2 "" H 5550 2750 50  0001 C CNN
@@
 P 7900 2150
 AR Path="/598183C5/5990A7F8" Ref="#PWR051"  Part="1"
-AR Path="/59933B07/5990A7F8" Ref="#PWR105"  Part="1"
-F 0 "#PWR051" H 7900 1900 50  0001 C CNN
+AR Path="/59933B07/5990A7F8" Ref="#PWR0108"  Part="1"
+F 0 "#PWR0108" H 7900 1900 50  0001 C CNN
 F 1 "GND" H 7900 2000 50  0000 C CNN
 F 2 "" H 7900 2150 50  0001 C CNN
@@
 P 3000 2250
 AR Path="/598183C5/5990A9E7" Ref="#PWR052"  Part="1"
-AR Path="/59933B07/5990A9E7" Ref="#PWR96"  Part="1"
-F 0 "#PWR052" H 3000 2000 50  0001 C CNN
+AR Path="/59933B07/5990A9E7" Ref="#PWR0109"  Part="1"
+F 0 "#PWR0109" H 3000 2000 50  0001 C CNN
 F 1 "GND" H 3000 2100 50  0000 C CNN
 F 2 "" H 3000 2250 50  0001 C CNN
@@
 P 5250 1700
 AR Path="/598183C5/5990AB6A" Ref="#PWR053"  Part="1"
-AR Path="/59933B07/5990AB6A" Ref="#PWR99"  Part="1"
-F 0 "#PWR053" H 5250 1550 50  0001 C CNN
+AR Path="/59933B07/5990AB6A" Ref="#PWR0110"  Part="1"
+F 0 "#PWR0110" H 5250 1550 50  0001 C CNN
 F 1 "VCC" H 5250 1850 50  0000 C CNN
 F 2 "" H 5250 1700 50  0001 C CNN
@@
 P 5450 1700
 AR Path="/598183C5/5990AB9B" Ref="#PWR054"  Part="1"
-AR Path="/59933B07/5990AB9B" Ref="#PWR101"  Part="1"
-F 0 "#PWR054" H 5450 1550 50  0001 C CNN
+AR Path="/59933B07/5990AB9B" Ref="#PWR0111"  Part="1"
+F 0 "#PWR0111" H 5450 1550 50  0001 C CNN
 F 1 "VCC" H 5450 1850 50  0000 C CNN
 F 2 "" H 5450 1700 50  0001 C CNN
@@
 AR Path="/598183C5/5992F278" Ref="U7"  Part="1"
 AR Path="/59933B07/5992F278" Ref="U11"  Part="1"
-F 0 "U7" H 5750 2900 60  0000 C CNN
+F 0 "U11" H 5750 2900 60  0000 C CNN
 F 1 "LH1526" H 5750 2750 60  0000 C CNN
 F 2 "" H 5750 2750 60  0001 C CNN

Commit message: Re-annotation
Parts:
- removed J7: CONN_01X05, symbol CONN_01X05
- removed unit 2 of U6
- added J10: CONN_01X05, symbol CONN_01X05
- added unit 2 of U9
- renumbered J6 to J9, U7 to U10, U6 to U9
Connections:
- net +3V3: now also U9.13 (V+)
- net GND: now also J10.2 (P2), U9.4 (V-), U9.5 (GND)
- net VCC: now also U9.12 (VCC)
- net prb1_b: now also U9.7 (IN)
- net prb2_a: now also J10.3 (P3)
- net prb2_b: now also J10.4 (P4)
- net prb2_v: now also J10.1 (P1)
- net prb3_rs_ctrl: now also U9.8 (SW)
- net vaisala_rs485_b: now also U9.6 (OUT)
Changed lines of the file:
@@
 $EndDescr
 $Comp
-L DG411 U6
+L DG411 U9
 U 1 1 5981A21D
 P 2300 4450
-AR Path="/598183C5/5981A21D" Ref="U6"  Part="1"
-AR Path="/59933B07/5981A21D" Ref="U10"  Part="1"
-F 0 "U10" H 2300 4550 50  0000 C CNN
+F 0 "U9" H 2300 4550 50  0000 C CNN
 F 1 "DG411" H 2300 4350 50  0000 C CNN
 F 2 "" H 2300 4450 60  0001 C CNN
@@
 $EndComp
 $Comp
-L GND #PWR041
-U 1 1 5981A4AC
+L GND #PWR92
+U 1 1 59945E5E
 P 2350 4950
-AR Path="/598183C5/5981A4AC" Ref="#PWR041"  Part="1"
-AR Path="/59933B07/5981A4AC" Ref="#PWR098"  Part="1"
-F 0 "#PWR098" H 2350 4700 50  0001 C CNN
+F 0 "#PWR92" H 2350 4700 50  0001 C CNN
 F 1 "GND" H 2350 4800 50  0000 C CNN
 F 2 "" H 2350 4950 50  0001 C CNN
@@
 $EndComp
 $Comp
-L GND #PWR042
-U 1 1 5981A5BD
+L GND #PWR95
+U 1 1 59945E5F
 P 4700 4950
-AR Path="/598183C5/5981A5BD" Ref="#PWR042"  Part="1"
-AR Path="/59933B07/5981A5BD" Ref="#PWR099"  Part="1"
-F 0 "#PWR099" H 4700 4700 50  0001 C CNN
+F 0 "#PWR95" H 4700 4700 50  0001 C CNN
 F 1 "GND" H 4700 4800 50  0000 C CNN
 F 2 "" H 4700 4950 50  0001 C CNN
@@
 $EndComp
 $Comp
-L +3.3V #PWR043
-U 1 1 5981A680
+L +3.3V #PWR91
+U 1 1 59945E60
 P 2350 3950
-AR Path="/598183C5/5981A680" Ref="#PWR043"  Part="1"
-AR Path="/59933B07/5981A680" Ref="#PWR0100"  Part="1"
-F 0 "#PWR0100" H 2350 3800 50  0001 C CNN
+F 0 "#PWR91" H 2350 3800 50  0001 C CNN
 F 1 "+3.3V" H 2350 4090 50  0000 C CNN
 F 2 "" H 2350 3950 50  0001 C CNN
@@
 $EndComp
 $Comp
-L +3.3V #PWR044
-U 1 1 5981A69E
+L +3.3V #PWR94
+U 1 1 59945E61
 P 4700 3950
-AR Path="/598183C5/5981A69E" Ref="#PWR044"  Part="1"
-AR Path="/59933B07/5981A69E" Ref="#PWR0101"  Part="1"
-F 0 "#PWR0101" H 4700 3800 50  0001 C CNN
+F 0 "#PWR94" H 4700 3800 50  0001 C CNN
 F 1 "+3.3V" H 4700 4090 50  0000 C CNN
 F 2 "" H 4700 3950 50  0001 C CNN
@@
 prb1_b
 $Comp
-L DG411 U6
-U 2 1 5981A26A
+L DG411 U9
+U 2 1 59945E5D
 P 4650 4450
-AR Path="/598183C5/5981A26A" Ref="U6"  Part="2"
-AR Path="/59933B07/5981A26A" Ref="U10"  Part="2"
-F 0 "U10" H 4650 4550 50  0000 C CNN
+F 0 "U9" H 4650 4550 50  0000 C CNN
 F 1 "DG411" H 4650 4350 50  0000 C CNN
 F 2 "" H 4650 4450 60  0001 C CNN
@@
 vaisala_rs485_b
 $Comp
-L DG411 U6
+L DG411 U9
 U 3 1 5981EAC3
 P 7400 4450
-AR Path="/598183C5/5981EAC3" Ref="U6"  Part="3"
-AR Path="/59933B07/5981EAC3" Ref="U10"  Part="3"
-F 0 "U10" H 7400 4550 50  0000 C CNN
+F 0 "U9" H 7400 4550 50  0000 C CNN
 F 1 "DG411" H 7400 4350 50  0000 C CNN
 F 2 "" H 7400 4450 60  0001 C CNN
@@
 $EndComp
 $Comp
-L GND #PWR045
+L GND #PWR101
 U 1 1 5981EAC9
 P 7450 4950
-AR Path="/598183C5/5981EAC9" Ref="#PWR045"  Part="1"
-AR Path="/59933B07/5981EAC9" Ref="#PWR0102"  Part="1"
-F 0 "#PWR0102" H 7450 4700 50  0001 C CNN
+F 0 "#PWR101" H 7450 4700 50  0001 C CNN
 F 1 "GND" H 7450 4800 50  0000 C CNN
 F 2 "" H 7450 4950 50  0001 C CNN
@@
 $EndComp
 $Comp
-L GND #PWR046
+L GND #PWR104
 U 1 1 5981EACF
 P 9500 4900
-AR Path="/598183C5/5981EACF" Ref="#PWR046"  Part="1"
-AR Path="/59933B07/5981EACF" Ref="#PWR0103"  Part="1"
-F 0 "#PWR0103" H 9500 4650 50  0001 C CNN
+F 0 "#PWR104" H 9500 4650 50  0001 C CNN
 F 1 "GND" H 9500 4750 50  0000 C CNN
 F 2 "" H 9500 4900 50  0001 C CNN
@@
 $EndComp
 $Comp
-L +3.3V #PWR047
+L +3.3V #PWR100
 U 1 1 5981EAD5
 P 7450 3950
-AR Path="/598183C5/5981EAD5" Ref="#PWR047"  Part="1"
-AR Path="/59933B07/5981EAD5" Ref="#PWR0104"  Part="1"
-F 0 "#PWR0104" H 7450 3800 50  0001 C CNN
+F 0 "#PWR100" H 7450 3800 50  0001 C CNN
 F 1 "+3.3V" H 7450 4090 50  0000 C CNN
 F 2 "" H 7450 3950 50  0001 C CNN
@@
 $EndComp
 $Comp
-L +3.3V #PWR048
+L +3.3V #PWR103
 U 1 1 5981EADB
 P 9500 3900
-AR Path="/598183C5/5981EADB" Ref="#PWR048"  Part="1"
-AR Path="/59933B07/5981EADB" Ref="#PWR0105"  Part="1"
-F 0 "#PWR0105" H 9500 3750 50  0001 C CNN
+F 0 "#PWR103" H 9500 3750 50  0001 C CNN
 F 1 "+3.3V" H 9500 4040 50  0000 C CNN
 F 2 "" H 9500 3900 50  0001 C CNN
@@
 prb2_b
 $Comp
-L DG411 U6
+L DG411 U9
 U 4 1 5981EAE3
 P 9450 4400
-AR Path="/598183C5/5981EAE3" Ref="U6"  Part="4"
-AR Path="/59933B07/5981EAE3" Ref="U10"  Part="4"
-F 0 "U10" H 9450 4500 50  0000 C CNN
+F 0 "U9" H 9450 4500 50  0000 C CNN
 F 1 "DG411" H 9450 4300 50  0000 C CNN
 F 2 "" H 9450 4400 60  0001 C CNN
@@
 vaisala_rs485_b
 $Comp
-L CONN_01X05 J6
+L CONN_01X05 J9
 U 1 1 598215F3
 P 3100 1700
-AR Path="/598183C5/598215F3" Ref="J6"  Part="1"
-AR Path="/59933B07/598215F3" Ref="J9"  Part="1"
 F 0 "J9" H 3100 2000 50  0000 C CNN
 F 1 "CONN_01X05" V 3200 1700 50  0000 C CNN
@@
 prb4_pwr_ctrl
 $Comp
-L CONN_01X05 J7
-U 1 1 59821868
+L CONN_01X05 J10
+U 1 1 59945E75
 P 8000 1600
-AR Path="/598183C5/59821868" Ref="J7"  Part="1"
-AR Path="/59933B07/59821868" Ref="J10"  Part="1"
 F 0 "J10" H 8000 1900 50  0000 C CNN
 F 1 "CONN_01X05" V 8100 1600 50  0000 C CNN
@@
 NoConn ~ 8200 1800
 $Comp
-L GND #PWR049
-U 1 1 5990A260
+L GND #PWR97
+U 1 1 59945E8B
 P 5350 2750
-AR Path="/598183C5/5990A260" Ref="#PWR049"  Part="1"
-AR Path="/59933B07/5990A260" Ref="#PWR0106"  Part="1"
-F 0 "#PWR0106" H 5350 2500 50  0001 C CNN
+F 0 "#PWR97" H 5350 2500 50  0001 C CNN
 F 1 "GND" H 5350 2600 50  0000 C CNN
 F 2 "" H 5350 2750 50  0001 C CNN
@@
 $EndComp
 $Comp
-L GND #PWR050
+L GND #PWR99
 U 1 1 5990A28D
 P 5550 2750
-AR Path="/598183C5/5990A28D" Ref="#PWR050"  Part="1"
-AR Path="/59933B07/5990A28D" Ref="#PWR0107"  Part="1"
-F 0 "#PWR0107" H 5550 2500 50  0001 C CNN
+F 0 "#PWR99" H 5550 2500 50  0001 C CNN
 F 1 "GND" H 5550 2600 50  0000 C CNN
 F 2 "" H 5550 2750 50  0001 C CNN
@@
 prb2_a
 $Comp
-L GND #PWR051
+L GND #PWR102
 U 1 1 5990A7F8
 P 7900 2150
-AR Path="/598183C5/5990A7F8" Ref="#PWR051"  Part="1"
-AR Path="/59933B07/5990A7F8" Ref="#PWR0108"  Part="1"
-F 0 "#PWR0108" H 7900 1900 50  0001 C CNN
+F 0 "#PWR102" H 7900 1900 50  0001 C CNN
 F 1 "GND" H 7900 2000 50  0000 C CNN
 F 2 "" H 7900 2150 50  0001 C CNN
@@
 $EndComp
 $Comp
-L GND #PWR052
-U 1 1 5990A9E7
+L GND #PWR93
+U 1 1 59945E8E
 P 3000 2250
-AR Path="/598183C5/5990A9E7" Ref="#PWR052"  Part="1"
-AR Path="/59933B07/5990A9E7" Ref="#PWR0109"  Part="1"
-F 0 "#PWR0109" H 3000 2000 50  0001 C CNN
+F 0 "#PWR93" H 3000 2000 50  0001 C CNN
 F 1 "GND" H 3000 2100 50  0000 C CNN
 F 2 "" H 3000 2250 50  0001 C CNN
@@
 $EndComp
 $Comp
-L VCC #PWR053
+L VCC #PWR96
 U 1 1 5990AB6A
 P 5250 1700
-AR Path="/598183C5/5990AB6A" Ref="#PWR053"  Part="1"
-AR Path="/59933B07/5990AB6A" Ref="#PWR0110"  Part="1"
-F 0 "#PWR0110" H 5250 1550 50  0001 C CNN
+F 0 "#PWR96" H 5250 1550 50  0001 C CNN
 F 1 "VCC" H 5250 1850 50  0000 C CNN
 F 2 "" H 5250 1700 50  0001 C CNN
@@
 $EndComp
 $Comp
-L VCC #PWR054
+L VCC #PWR98
 U 1 1 5990AB9B
 P 5450 1700
-AR Path="/598183C5/5990AB9B" Ref="#PWR054"  Part="1"
-AR Path="/59933B07/5990AB9B" Ref="#PWR0111"  Part="1"
-F 0 "#PWR0111" H 5450 1550 50  0001 C CNN
+F 0 "#PWR98" H 5450 1550 50  0001 C CNN
 F 1 "VCC" H 5450 1850 50  0000 C CNN
 F 2 "" H 5450 1700 50  0001 C CNN
@@
 prb2_v
 $Comp
-L LH1526 U7
+L LH1526 U10
 U 1 1 5992F278
 P 5700 2800
-AR Path="/598183C5/5992F278" Ref="U7"  Part="1"
-AR Path="/59933B07/5992F278" Ref="U11"  Part="1"
-F 0 "U11" H 5750 2900 60  0000 C CNN
+F 0 "U10" H 5750 2900 60  0000 C CNN
 F 1 "LH1526" H 5750 2750 60  0000 C CNN
 F 2 "" H 5750 2750 60  0001 C CNN
