File: probe_module2.sch (KiCad schematic (older format))
At the start: 4 parts, among them J10 M12, J9 M12, U10 LH1526, U9 DG411

Commit message: fix footprint errors
Parts:
- U9: footprint Housings_SOIC:SOIC-8_3.9x4.9mm_Pitch1.27mm -> Housings_DIP:DIP-16_W7.62mm_SMD
Changed lines of the file:
@@
 F 0 "U9" H 2300 4550 50  0000 C CNN
 F 1 "DG411" H 2300 4350 50  0000 C CNN
-F 2 "Housings_SOIC:SOIC-8_3.9x4.9mm_Pitch1.27mm" H 2300 4450 60  0001 C CNN
+F 2 "Housings_DIP:DIP-16_W7.62mm_SMD" H 2300 4450 60  0001 C CNN
 F 3 "" H 2300 4450 60  0001 C CNN
 	1    2300 4450
@@
 F 0 "U9" H 4650 4550 50  0000 C CNN
 F 1 "DG411" H 4650 4350 50  0000 C CNN
-F 2 "Housings_SOIC:SOIC-8_3.9x4.9mm_Pitch1.27mm" H 4650 4450 60  0001 C CNN
+F 2 "Housings_DIP:DIP-16_W7.62mm_SMD" H 4650 4450 60  0001 C CNN
 F 3 "" H 4650 4450 60  0001 C CNN
 	2    4650 4450
@@
 F 0 "U9" H 7400 4550 50  0000 C CNN
 F 1 "DG411" H 7400 4350 50  0000 C CNN
-F 2 "Housings_SOIC:SOIC-8_3.9x4.9mm_Pitch1.27mm" H 7400 4450 60  0001 C CNN
+F 2 "Housings_DIP:DIP-16_W7.62mm_SMD" H 7400 4450 60  0001 C CNN
 F 3 "" H 7400 4450 60  0001 C CNN
 	3    7400 4450
@@
 F 0 "U9" H 9450 4500 50  0000 C CNN
 F 1 "DG411" H 9450 4300 50  0000 C CNN
-F 2 "Housings_SOIC:SOIC-8_3.9x4.9mm_Pitch1.27mm" H 9450 4400 60  0001 C CNN
+F 2 "Housings_DIP:DIP-16_W7.62mm_SMD" H 9450 4400 60  0001 C CNN
 F 3 "" H 9450 4400 60  0001 C CNN
 	4    9450 4400
