File: pt-module-interface4.sch (KiCad schematic (older format))
At the start: 8 parts, among them SW2 SW_Push, SW3 SW_Push

Commit message: Connected EVERYTHING. Ran ERC. There are still some power errors.
Connections:
- net prb1_pwr_btn renamed prb4_pwr_btn
- net prb1_pwr_led_in renamed prb4_pwr_led_in
- net prb1_rs_btn renamed prb4_rs_btn
- net prb1_rs_led_in renamed prb4_rs_led_in
Changed lines of the file:
@@
 $Descr A4 11693 8268
 encoding utf-8
-Sheet 5 13
+Sheet 12 13
 Title ""
 Date ""
@@
 AR Path="/598B3EA9/598198A0" Ref="D15"  Part="1"
 AR Path="/598B41A3/598198A0" Ref="D17"  Part="1"
-F 0 "D11" H 2600 2600 50  0000 C CNN
+F 0 "D17" H 2600 2600 50  0000 C CNN
 F 1 "LED" H 2600 2400 50  0000 C CNN
 F 2 "" H 2600 2500 50  0001 C CNN
@@
 AR Path="/598B3EA9/598199D3" Ref="SW6"  Part="1"
 AR Path="/598B41A3/598199D3" Ref="SW12"  Part="1"
-F 0 "SW2" H 2650 3650 50  0000 L CNN
+F 0 "SW12" H 2650 3650 50  0000 L CNN
 F 1 "SW_Push" H 2600 3490 50  0000 C CNN
 F 2 "" H 2600 3750 50  0001 C CNN
@@
 AR Path="/598B3EA9/59819AA1" Ref="R20"  Part="1"
 AR Path="/598B41A3/59819AA1" Ref="R28"  Part="1"
-F 0 "R12" V 3130 2500 50  0000 C CNN
+F 0 "R28" V 3130 2500 50  0000 C CNN
 F 1 "1k8" V 3050 2500 50  0000 C CNN
 F 2 "" V 2980 2500 50  0001 C CNN
@@
 AR Path="/598B3EA9/5981A7B1" Ref="R19"  Part="1"
 AR Path="/598B41A3/5981A7B1" Ref="R27"  Part="1"
-F 0 "R11" V 2980 3250 50  0000 C CNN
+F 0 "R27" V 2980 3250 50  0000 C CNN
 F 1 "10k" V 2900 3250 50  0000 C CNN
 F 2 "" V 2830 3250 50  0001 C CNN
@@
 P 2900 3100
 AR Path="/59819805/5981A7F0" Ref="#PWR055"  Part="1"
-AR Path="/598B38EB/5981A7F0" Ref="#PWR65"  Part="1"
-AR Path="/598B3EA9/5981A7F0" Ref="#PWR71"  Part="1"
-AR Path="/598B41A3/5981A7F0" Ref="#PWR90"  Part="1"
-F 0 "#PWR055" H 2900 2950 50  0001 C CNN
+AR Path="/598B38EB/5981A7F0" Ref="#PWR067"  Part="1"
+AR Path="/598B3EA9/5981A7F0" Ref="#PWR073"  Part="1"
+AR Path="/598B41A3/5981A7F0" Ref="#PWR092"  Part="1"
+F 0 "#PWR092" H 2900 2950 50  0001 C CNN
 F 1 "+3.3V" H 2900 3240 50  0000 C CNN
 F 2 "" H 2900 3100 50  0001 C CNN
@@
 P 2200 3600
 AR Path="/59819805/5981A91C" Ref="#PWR056"  Part="1"
-AR Path="/598B38EB/5981A91C" Ref="#PWR63"  Part="1"
-AR Path="/598B3EA9/5981A91C" Ref="#PWR69"  Part="1"
-AR Path="/598B41A3/5981A91C" Ref="#PWR88"  Part="1"
-F 0 "#PWR056" H 2200 3350 50  0001 C CNN
+AR Path="/598B38EB/5981A91C" Ref="#PWR068"  Part="1"
+AR Path="/598B3EA9/5981A91C" Ref="#PWR074"  Part="1"
+AR Path="/598B41A3/5981A91C" Ref="#PWR093"  Part="1"
+F 0 "#PWR093" H 2200 3350 50  0001 C CNN
 F 1 "GND" H 2200 3450 50  0000 C CNN
 F 2 "" H 2200 3600 50  0001 C CNN
@@
 $EndComp
 Text HLabel 3050 3550 2    60   Input ~ 0
-prb1_pwr_btn
+prb4_pwr_btn
 $Comp
 L GND #PWR057
@@
 P 2300 2600
 AR Path="/59819805/5981B0C2" Ref="#PWR057"  Part="1"
-AR Path="/598B38EB/5981B0C2" Ref="#PWR64"  Part="1"
-AR Path="/598B3EA9/5981B0C2" Ref="#PWR70"  Part="1"
-AR Path="/598B41A3/5981B0C2" Ref="#PWR89"  Part="1"
-F 0 "#PWR057" H 2300 2350 50  0001 C CNN
+AR Path="/598B38EB/5981B0C2" Ref="#PWR069"  Part="1"
+AR Path="/598B3EA9/5981B0C2" Ref="#PWR075"  Part="1"
+AR Path="/598B41A3/5981B0C2" Ref="#PWR094"  Part="1"
+F 0 "#PWR094" H 2300 2350 50  0001 C CNN
 F 1 "GND" H 2300 2450 50  0000 C CNN
 F 2 "" H 2300 2600 50  0001 C CNN
@@
 $EndComp
 Text HLabel 3300 2500 2    60   Input ~ 0
-prb1_pwr_led_in
+prb4_pwr_led_in
 Wire Wire Line
 	2800 3550 3050 3550
@@
 	2900 3400 2900 3550
 Text HLabel 5200 3600 2    60   Input ~ 0
-prb1_rs_btn
+prb4_rs_btn
 $Comp
 L SW_Push SW3
@@
 AR Path="/598B3EA9/59898241" Ref="SW7"  Part="1"
 AR Path="/598B41A3/59898241" Ref="SW13"  Part="1"
-F 0 "SW3" H 4800 3700 50  0000 L CNN
+F 0 "SW13" H 4800 3700 50  0000 L CNN
 F 1 "SW_Push" H 4750 3540 50  0000 C CNN
 F 2 "" H 4750 3800 50  0001 C CNN
@@
 AR Path="/598B3EA9/59898247" Ref="R21"  Part="1"
 AR Path="/598B41A3/59898247" Ref="R29"  Part="1"
-F 0 "R13" V 5130 3300 50  0000 C CNN
+F 0 "R29" V 5130 3300 50  0000 C CNN
 F 1 "10k" V 5050 3300 50  0000 C CNN
 F 2 "" V 4980 3300 50  0001 C CNN
@@
 P 5050 3150
 AR Path="/59819805/5989824D" Ref="#PWR058"  Part="1"
-AR Path="/598B38EB/5989824D" Ref="#PWR68"  Part="1"
-AR Path="/598B3EA9/5989824D" Ref="#PWR74"  Part="1"
-AR Path="/598B41A3/5989824D" Ref="#PWR93"  Part="1"
-F 0 "#PWR058" H 5050 3000 50  0001 C CNN
+AR Path="/598B38EB/5989824D" Ref="#PWR070"  Part="1"
+AR Path="/598B3EA9/5989824D" Ref="#PWR076"  Part="1"
+AR Path="/598B41A3/5989824D" Ref="#PWR095"  Part="1"
+F 0 "#PWR095" H 5050 3000 50  0001 C CNN
 F 1 "+3.3V" H 5050 3290 50  0000 C CNN
 F 2 "" H 5050 3150 50  0001 C CNN
@@
 P 4350 3650
 AR Path="/59819805/59898253" Ref="#PWR059"  Part="1"
-AR Path="/598B38EB/59898253" Ref="#PWR66"  Part="1"
-AR Path="/598B3EA9/59898253" Ref="#PWR72"  Part="1"
-AR Path="/598B41A3/59898253" Ref="#PWR91"  Part="1"
-F 0 "#PWR059" H 4350 3400 50  0001 C CNN
+AR Path="/598B38EB/59898253" Ref="#PWR071"  Part="1"
+AR Path="/598B3EA9/59898253" Ref="#PWR077"  Part="1"
+AR Path="/598B41A3/59898253" Ref="#PWR096"  Part="1"
+F 0 "#PWR096" H 4350 3400 50  0001 C CNN
 F 1 "GND" H 4350 3500 50  0000 C CNN
 F 2 "" H 4350 3650 50  0001 C CNN
@@
 AR Path="/598B3EA9/598986C7" Ref="D16"  Part="1"
 AR Path="/598B41A3/598986C7" Ref="D18"  Part="1"
-F 0 "D12" H 4900 2600 50  0000 C CNN
+F 0 "D18" H 4900 2600 50  0000 C CNN
 F 1 "LED" H 4900 2400 50  0000 C CNN
 F 2 "" H 4900 2500 50  0001 C CNN
@@
 AR Path="/598B3EA9/598986CD" Ref="R22"  Part="1"
 AR Path="/598B41A3/598986CD" Ref="R30"  Part="1"
-F 0 "R14" V 5430 2500 50  0000 C CNN
+F 0 "R30" V 5430 2500 50  0000 C CNN
 F 1 "1k8" V 5350 2500 50  0000 C CNN
 F 2 "" V 5280 2500 50  0001 C CNN
@@
 P 4600 2600
 AR Path="/59819805/598986D3" Ref="#PWR060"  Part="1"
-AR Path="/598B38EB/598986D3" Ref="#PWR67"  Part="1"
-AR Path="/598B3EA9/598986D3" Ref="#PWR73"  Part="1"
-AR Path="/598B41A3/598986D3" Ref="#PWR92"  Part="1"
-F 0 "#PWR060" H 4600 2350 50  0001 C CNN
+AR Path="/598B38EB/598986D3" Ref="#PWR072"  Part="1"
+AR Path="/598B3EA9/598986D3" Ref="#PWR078"  Part="1"
+AR Path="/598B41A3/598986D3" Ref="#PWR097"  Part="1"
+F 0 "#PWR097" H 4600 2350 50  0001 C CNN
 F 1 "GND" H 4600 2450 50  0000 C CNN
 F 2 "" H 4600 2600 50  0001 C CNN
@@
 	4750 2500 4600 2500
 Text HLabel 5600 2500 2    60   Input ~ 0
-prb1_rs_led_in
+prb4_rs_led_in
 $EndSCHEMATC

Commit message: Re-annotation
Parts:
- removed D11, D12: LED, symbol LED
- removed R13: 10k, symbol R
- removed R14: 1k8, symbol R
- removed SW2, SW3: SW_Push, symbol SW_Push
- added D14, D15: LED, symbol LED
- added R31: 10k, symbol R
- added R32: 1k8, symbol R
- added SW12, SW13: SW_Push, symbol SW_Push
- renumbered R11 to R29, R12 to R30
Connections:
- net +3V3: now also R31.2
- net GND: now also D14.1 (K), D15.1 (K), SW12.1, SW13.1
- net prb4_pwr_btn: now also SW12.2
- net prb4_rs_btn: now also R31.1, SW13.2
- net prb4_rs_led_in: now also R32.1
- net at R30.2: now also D14.2 (A)
- new net: D15.2 (A), R32.2
Changed lines of the file:
@@
 $EndDescr
 $Comp
-L LED D11
-U 1 1 598198A0
+L LED D14
+U 1 1 59945E54
 P 2600 2500
-AR Path="/59819805/598198A0" Ref="D11"  Part="1"
-AR Path="/598B38EB/598198A0" Ref="D13"  Part="1"
-AR Path="/598B3EA9/598198A0" Ref="D15"  Part="1"
-AR Path="/598B41A3/598198A0" Ref="D17"  Part="1"
-F 0 "D17" H 2600 2600 50  0000 C CNN
+F 0 "D14" H 2600 2600 50  0000 C CNN
 F 1 "LED" H 2600 2400 50  0000 C CNN
 F 2 "" H 2600 2500 50  0001 C CNN
@@
 $EndComp
 $Comp
-L SW_Push SW2
-U 1 1 598199D3
+L SW_Push SW12
+U 1 1 59945E58
 P 2600 3550
-AR Path="/59819805/598199D3" Ref="SW2"  Part="1"
-AR Path="/598B38EB/598199D3" Ref="SW4"  Part="1"
-AR Path="/598B3EA9/598199D3" Ref="SW6"  Part="1"
-AR Path="/598B41A3/598199D3" Ref="SW12"  Part="1"
 F 0 "SW12" H 2650 3650 50  0000 L CNN
 F 1 "SW_Push" H 2600 3490 50  0000 C CNN
@@
 $EndComp
 $Comp
-L R R12
+L R R30
 U 1 1 59819AA1
 P 3050 2500
-AR Path="/59819805/59819AA1" Ref="R12"  Part="1"
-AR Path="/598B38EB/59819AA1" Ref="R16"  Part="1"
-AR Path="/598B3EA9/59819AA1" Ref="R20"  Part="1"
-AR Path="/598B41A3/59819AA1" Ref="R28"  Part="1"
-F 0 "R28" V 3130 2500 50  0000 C CNN
+F 0 "R30" V 3130 2500 50  0000 C CNN
 F 1 "1k8" V 3050 2500 50  0000 C CNN
 F 2 "" V 2980 2500 50  0001 C CNN
@@
 $EndComp
 $Comp
-L R R11
+L R R29
 U 1 1 5981A7B1
 P 2900 3250
-AR Path="/59819805/5981A7B1" Ref="R11"  Part="1"
-AR Path="/598B38EB/5981A7B1" Ref="R15"  Part="1"
-AR Path="/598B3EA9/5981A7B1" Ref="R19"  Part="1"
-AR Path="/598B41A3/5981A7B1" Ref="R27"  Part="1"
-F 0 "R27" V 2980 3250 50  0000 C CNN
+F 0 "R29" V 2980 3250 50  0000 C CNN
 F 1 "10k" V 2900 3250 50  0000 C CNN
 F 2 "" V 2830 3250 50  0001 C CNN
@@
 $EndComp
 $Comp
-L +3.3V #PWR055
+L +3.3V #PWR87
 U 1 1 5981A7F0
 P 2900 3100
-AR Path="/59819805/5981A7F0" Ref="#PWR055"  Part="1"
-AR Path="/598B38EB/5981A7F0" Ref="#PWR067"  Part="1"
-AR Path="/598B3EA9/5981A7F0" Ref="#PWR073"  Part="1"
-AR Path="/598B41A3/5981A7F0" Ref="#PWR092"  Part="1"
-F 0 "#PWR092" H 2900 2950 50  0001 C CNN
+F 0 "#PWR87" H 2900 2950 50  0001 C CNN
 F 1 "+3.3V" H 2900 3240 50  0000 C CNN
 F 2 "" H 2900 3100 50  0001 C CNN
@@
 $EndComp
 $Comp
-L GND #PWR056
+L GND #PWR85
 U 1 1 5981A91C
 P 2200 3600
-AR Path="/59819805/5981A91C" Ref="#PWR056"  Part="1"
-AR Path="/598B38EB/5981A91C" Ref="#PWR068"  Part="1"
-AR Path="/598B3EA9/5981A91C" Ref="#PWR074"  Part="1"
-AR Path="/598B41A3/5981A91C" Ref="#PWR093"  Part="1"
-F 0 "#PWR093" H 2200 3350 50  0001 C CNN
+F 0 "#PWR85" H 2200 3350 50  0001 C CNN
 F 1 "GND" H 2200 3450 50  0000 C CNN
 F 2 "" H 2200 3600 50  0001 C CNN
@@
 prb4_pwr_btn
 $Comp
-L GND #PWR057
-U 1 1 5981B0C2
+L GND #PWR86
+U 1 1 59945E6D
 P 2300 2600
-AR Path="/59819805/5981B0C2" Ref="#PWR057"  Part="1"
-AR Path="/598B38EB/5981B0C2" Ref="#PWR069"  Part="1"
-AR Path="/598B3EA9/5981B0C2" Ref="#PWR075"  Part="1"
-AR Path="/598B41A3/5981B0C2" Ref="#PWR094"  Part="1"
-F 0 "#PWR094" H 2300 2350 50  0001 C CNN
+F 0 "#PWR86" H 2300 2350 50  0001 C CNN
 F 1 "GND" H 2300 2450 50  0000 C CNN
 F 2 "" H 2300 2600 50  0001 C CNN
@@
 prb4_rs_btn
 $Comp
-L SW_Push SW3
-U 1 1 59898241
+L SW_Push SW13
+U 1 1 59945E77
 P 4750 3600
-AR Path="/59819805/59898241" Ref="SW3"  Part="1"
-AR Path="/598B38EB/59898241" Ref="SW5"  Part="1"
-AR Path="/598B3EA9/59898241" Ref="SW7"  Part="1"
-AR Path="/598B41A3/59898241" Ref="SW13"  Part="1"
 F 0 "SW13" H 4800 3700 50  0000 L CNN
 F 1 "SW_Push" H 4750 3540 50  0000 C CNN
@@
 $EndComp
 $Comp
-L R R13
-U 1 1 59898247
+L R R31
+U 1 1 59945E79
 P 5050 3300
-AR Path="/59819805/59898247" Ref="R13"  Part="1"
-AR Path="/598B38EB/59898247" Ref="R17"  Part="1"
-AR Path="/598B3EA9/59898247" Ref="R21"  Part="1"
-AR Path="/598B41A3/59898247" Ref="R29"  Part="1"
-F 0 "R29" V 5130 3300 50  0000 C CNN
+F 0 "R31" V 5130 3300 50  0000 C CNN
 F 1 "10k" V 5050 3300 50  0000 C CNN
 F 2 "" V 4980 3300 50  0001 C CNN
@@
 $EndComp
 $Comp
-L +3.3V #PWR058
-U 1 1 5989824D
+L +3.3V #PWR90
+U 1 1 59945E7D
 P 5050 3150
-AR Path="/59819805/5989824D" Ref="#PWR058"  Part="1"
-AR Path="/598B38EB/5989824D" Ref="#PWR070"  Part="1"
-AR Path="/598B3EA9/5989824D" Ref="#PWR076"  Part="1"
-AR Path="/598B41A3/5989824D" Ref="#PWR095"  Part="1"
-F 0 "#PWR095" H 5050 3000 50  0001 C CNN
+F 0 "#PWR90" H 5050 3000 50  0001 C CNN
 F 1 "+3.3V" H 5050 3290 50  0000 C CNN
 F 2 "" H 5050 3150 50  0001 C CNN
@@
 $EndComp
 $Comp
-L GND #PWR059
-U 1 1 59898253
+L GND #PWR88
+U 1 1 59945E7F
 P 4350 3650
-AR Path="/59819805/59898253" Ref="#PWR059"  Part="1"
-AR Path="/598B38EB/59898253" Ref="#PWR071"  Part="1"
-AR Path="/598B3EA9/59898253" Ref="#PWR077"  Part="1"
-AR Path="/598B41A3/59898253" Ref="#PWR096"  Part="1"
-F 0 "#PWR096" H 4350 3400 50  0001 C CNN
+F 0 "#PWR88" H 4350 3400 50  0001 C CNN
 F 1 "GND" H 4350 3500 50  0000 C CNN
 F 2 "" H 4350 3650 50  0001 C CNN
@@
 	5050 3450 5050 3600
 $Comp
-L LED D12
-U 1 1 598986C7
+L LED D15
+U 1 1 59945E84
 P 4900 2500
-AR Path="/59819805/598986C7" Ref="D12"  Part="1"
-AR Path="/598B38EB/598986C7" Ref="D14"  Part="1"
-AR Path="/598B3EA9/598986C7" Ref="D16"  Part="1"
-AR Path="/598B41A3/598986C7" Ref="D18"  Part="1"
-F 0 "D18" H 4900 2600 50  0000 C CNN
+F 0 "D15" H 4900 2600 50  0000 C CNN
 F 1 "LED" H 4900 2400 50  0000 C CNN
 F 2 "" H 4900 2500 50  0001 C CNN
@@
 $EndComp
 $Comp
-L R R14
-U 1 1 598986CD
+L R R32
+U 1 1 59945E87
 P 5350 2500
-AR Path="/59819805/598986CD" Ref="R14"  Part="1"
-AR Path="/598B38EB/598986CD" Ref="R18"  Part="1"
-AR Path="/598B3EA9/598986CD" Ref="R22"  Part="1"
-AR Path="/598B41A3/598986CD" Ref="R30"  Part="1"
-F 0 "R30" V 5430 2500 50  0000 C CNN
+F 0 "R32" V 5430 2500 50  0000 C CNN
 F 1 "1k8" V 5350 2500 50  0000 C CNN
 F 2 "" V 5280 2500 50  0001 C CNN
@@
 $EndComp
 $Comp
-L GND #PWR060
+L GND #PWR89
 U 1 1 598986D3
 P 4600 2600
-AR Path="/59819805/598986D3" Ref="#PWR060"  Part="1"
-AR Path="/598B38EB/598986D3" Ref="#PWR072"  Part="1"
-AR Path="/598B3EA9/598986D3" Ref="#PWR078"  Part="1"
-AR Path="/598B41A3/598986D3" Ref="#PWR097"  Part="1"
-F 0 "#PWR097" H 4600 2350 50  0001 C CNN
+F 0 "#PWR89" H 4600 2350 50  0001 C CNN
 F 1 "GND" H 4600 2450 50  0000 C CNN
 F 2 "" H 4600 2600 50  0001 C CNN
