File: pt-module-interface4.sch (KiCad schematic (older format))
At the start: 8 parts, among them SW12 SW_Push, SW13 SW_Push

Commit message: add all the rest of the footprints
Parts:
- D14, D15, SW12, SW13: footprint (none) -> Connectors_Hirose:Hirose_DF13C-02P-1.25V_02x1.25mm_Straight
- R29, R30, R31, R32: footprint (none) -> Resistors_SMD:R_1206_HandSoldering
Changed lines of the file:
@@
 F 0 "D14" H 2600 2600 50  0000 C CNN
 F 1 "LED" H 2600 2400 50  0000 C CNN
-F 2 "" H 2600 2500 50  0001 C CNN
+F 2 "Connectors_Hirose:Hirose_DF13C-02P-1.25V_02x1.25mm_Straight" H 2600 2500 50  0001 C CNN
 F 3 "" H 2600 2500 50  0001 C CNN
 	1    2600 2500
@@
 F 0 "SW12" H 2650 3650 50  0000 L CNN
 F 1 "SW_Push" H 2600 3490 50  0000 C CNN
-F 2 "" H 2600 3750 50  0001 C CNN
+F 2 "Connectors_Hirose:Hirose_DF13C-02P-1.25V_02x1.25mm_Straight" H 2600 3750 50  0001 C CNN
 F 3 "" H 2600 3750 50  0001 C CNN
 	1    2600 3550
@@
 F 0 "R30" V 3130 2500 50  0000 C CNN
 F 1 "1k8" V 3050 2500 50  0000 C CNN
-F 2 "" V 2980 2500 50  0001 C CNN
+F 2 "Resistors_SMD:R_1206_HandSoldering" V 2980 2500 50  0001 C CNN
 F 3 "" H 3050 2500 50  0001 C CNN
 	1    3050 2500
@@
 F 0 "R29" V 2980 3250 50  0000 C CNN
 F 1 "10k" V 2900 3250 50  0000 C CNN
-F 2 "" V 2830 3250 50  0001 C CNN
+F 2 "Resistors_SMD:R_1206_HandSoldering" V 2830 3250 50  0001 C CNN
 F 3 "" H 2900 3250 50  0001 C CNN
 	1    2900 3250
@@
 F 0 "SW13" H 4800 3700 50  0000 L CNN
 F 1 "SW_Push" H 4750 3540 50  0000 C CNN
-F 2 "" H 4750 3800 50  0001 C CNN
+F 2 "Connectors_Hirose:Hirose_DF13C-02P-1.25V_02x1.25mm_Straight" H 4750 3800 50  0001 C CNN
 F 3 "" H 4750 3800 50  0001 C CNN
 	1    4750 3600
@@
 F 0 "R31" V 5130 3300 50  0000 C CNN
 F 1 "10k" V 5050 3300 50  0000 C CNN
-F 2 "" V 4980 3300 50  0001 C CNN
+F 2 "Resistors_SMD:R_1206_HandSoldering" V 4980 3300 50  0001 C CNN
 F 3 "" H 5050 3300 50  0001 C CNN
 	1    5050 3300
@@
 F 0 "D15" H 4900 2600 50  0000 C CNN
 F 1 "LED" H 4900 2400 50  0000 C CNN
-F 2 "" H 4900 2500 50  0001 C CNN
+F 2 "Connectors_Hirose:Hirose_DF13C-02P-1.25V_02x1.25mm_Straight" H 4900 2500 50  0001 C CNN
 F 3 "" H 4900 2500 50  0001 C CNN
 	1    4900 2500
@@
 F 0 "R32" V 5430 2500 50  0000 C CNN
 F 1 "1k8" V 5350 2500 50  0000 C CNN
-F 2 "" V 5280 2500 50  0001 C CNN
+F 2 "Resistors_SMD:R_1206_HandSoldering" V 5280 2500 50  0001 C CNN
 F 3 "" H 5350 2500 50  0001 C CNN
 	1    5350 2500
