File: pt-module-usb-interface.sch (KiCad schematic (older format))
At the start: 9 parts, among them J8 USB_OTG, U7 FT230XS

Commit message: add all the rest of the footprints
Parts:
- C11, C12, C13: footprint (none) -> Capacitors_SMD:C_1206_HandSoldering
- J8: footprint (none) -> Connectors_Hirose:Hirose_DF13C-06P-1.25V_06x1.25mm_Straight
- R13, R14, R15, R16: footprint (none) -> Resistors_SMD:R_1206_HandSoldering
Changed lines of the file:
@@
 F 0 "J8" H 3600 4650 50  0000 L CNN
 F 1 "USB_OTG" H 3600 4550 50  0000 L CNN
-F 2 "" H 3950 4150 50  0001 C CNN
+F 2 "Connectors_Hirose:Hirose_DF13C-06P-1.25V_06x1.25mm_Straight" H 3950 4150 50  0001 C CNN
 F 3 "" H 3950 4150 50  0001 C CNN
 	1    3800 4200
@@
 F 0 "R15" V 5680 4000 50  0000 C CNN
 F 1 "4k7" V 5600 4000 50  0000 C CNN
-F 2 "" V 5530 4000 50  0001 C CNN
+F 2 "Resistors_SMD:R_1206_HandSoldering" V 5530 4000 50  0001 C CNN
 F 3 "" H 5600 4000 50  0001 C CNN
 	1    5600 4000
@@
 F 0 "R16" V 5980 4200 50  0000 C CNN
 F 1 "10k" V 5900 4200 50  0000 C CNN
-F 2 "" V 5830 4200 50  0001 C CNN
+F 2 "Resistors_SMD:R_1206_HandSoldering" V 5830 4200 50  0001 C CNN
 F 3 "" H 5900 4200 50  0001 C CNN
 	1    5900 4200
@@
 F 0 "R13" V 4380 3000 50  0000 C CNN
 F 1 "27R" V 4300 3000 50  0000 C CNN
-F 2 "" V 4230 3000 50  0001 C CNN
+F 2 "Resistors_SMD:R_1206_HandSoldering" V 4230 3000 50  0001 C CNN
 F 3 "" H 4300 3000 50  0001 C CNN
 	1    4300 3000
@@
 F 0 "R14" V 4580 3000 50  0000 C CNN
 F 1 "27R" V 4500 3000 50  0000 C CNN
-F 2 "" V 4430 3000 50  0001 C CNN
+F 2 "Resistors_SMD:R_1206_HandSoldering" V 4430 3000 50  0001 C CNN
 F 3 "" H 4500 3000 50  0001 C CNN
 	1    4500 3000
@@
 F 0 "C11" H 4710 3520 50  0000 L CNN
 F 1 "47pF" H 4710 3370 50  0000 L CNN
-F 2 "" H 4700 3450 50  0001 C CNN
+F 2 "Capacitors_SMD:C_1206_HandSoldering" H 4700 3450 50  0001 C CNN
 F 3 "" H 4700 3450 50  0001 C CNN
 	1    4700 3450
@@
 F 0 "C12" H 4710 3820 50  0000 L CNN
 F 1 "47pF" H 4710 3670 50  0000 L CNN
-F 2 "" H 4700 3750 50  0001 C CNN
+F 2 "Capacitors_SMD:C_1206_HandSoldering" H 4700 3750 50  0001 C CNN
 F 3 "" H 4700 3750 50  0001 C CNN
 	1    4700 3750
@@
 F 0 "C13" H 4960 3270 50  0000 L CNN
 F 1 "100nF" H 4960 3120 50  0000 L CNN
-F 2 "" H 4950 3200 50  0001 C CNN
+F 2 "Capacitors_SMD:C_1206_HandSoldering" H 4950 3200 50  0001 C CNN
 F 3 "" H 4950 3200 50  0001 C CNN
 	1    4950 3200
