File: pt-module.kicad_pcb (KiCad board)
At the start: 2 copper layers, 107 parts, among them J1 M12 in, J10 M12, J2 Ethercon out, J3 PWR in, J4 M12 out, J5 Ethercon out, J6 M12, J7 M12, J8 USB_OTG, J9 M12, SW1 pwr-source switch, SW10 SW_Push, SW11 SW_Push, SW12 SW_Push, SW13 SW_Push, SW2 SW_Push, SW3 SW_Push, SW4 SW_Push, SW5 SW_Push, SW6 SW_Push, SW7 SW_Push, SW8 SW_Push, SW9 SW_Push, U1 MCP16331, U10 LH1526, U2 MCP16331, U3 SN65HVD72, U4 SN65HVD72, U5 DG411, U6 LH1526, U7 FT230XS, U8 STM32F334R8Tx, U9 DG411

Commit message: start the pcb
Parts:
- moved D8 128.2 mm to (53.3, 19.1), turned to 180 degrees
- moved R10 126.8 mm to (50.8, 24.1)
- moved D9 121.8 mm to (62.2, 19.1), turned to 180 degrees
- moved SW2 117.7 mm to (58.4, 29.2), turned to 180 degrees
- moved R12 117.3 mm to (63.5, 24.1), turned to 180 degrees
- moved J6 114.8 mm to (72.4, 19.1), turned to 180 degrees
- moved R9 113.7 mm to (58.4, 35.6)
- moved SW3 110.1 mm to (68.6, 29.2), turned to 180 degrees
- moved J4 109.0 mm to (247.7, 59.7), turned to 90 degrees
- moved D10 107.6 mm to (83.8, 19.1), turned to 180 degrees
- moved R11 105.9 mm to (68.6, 35.6)
- moved J2 102.6 mm to (247.7, 78.7), turned to 90 degrees
- moved D11 102.5 mm to (92.7, 19.1), turned to 180 degrees
- moved R17 100.3 mm to (80.0, 31.8), turned to 180 degrees
- moved R18 97.6 mm to (77.5, 38.1)
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
Commit message: pcb design
Parts:
- ?: renamed from 330R1; value R -> 330R
- ?: renamed from .1; footprint Housings_DIP:DIP-8_W11.48mm_SMD -> Housings_SOIC:SO-4_4.4x4.3mm_Pitch2.54mm
- moved R31 75.7 mm to (181.6, 29.2)
- moved C12 62.3 mm to (160.9, 88.4)
- moved J4 61.5 mm to (187.8, 74.2)
- moved 16Mhz1 61.1 mm to (138.0, 80.4), turned to 90 degrees
- moved J2 60.7 mm to (187.8, 88.8)
- moved C14 49.9 mm to (135.1, 88.7), turned to 270 degrees
- moved C10 49.6 mm to (168.9, 77.0), turned to 90 degrees
- moved C15 47.5 mm to (134.8, 75.5), turned to 90 degrees
- moved R3 45.9 mm to (83.8, 120.7), turned to 180 degrees
- moved D12 45.7 mm to (172.7, 19.1)
- moved D14 45.7 mm to (203.2, 19.1)
- moved D15 45.7 mm to (212.1, 19.1)
- moved C21 45.6 mm to (156.0, 102.4)
- moved D13 44.5 mm to (180.3, 19.1)
- moved J10 44.5 mm to (191.8, 19.1)
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- renumbered 120R1 to Terminator
Routing:
- net /PT module interface/prb1_rs_btn: track 0.00 -> 5.51 mm
- net Net-(D8-Pad2): track 0.00 -> 4.99 mm
- net /PT module interface/prb1_pwr_btn: track 0.00 -> 4.99 mm
- net +3V3: track 0.00 -> 2.35 mm

Commit message: Updated PCB
Parts:
- moved U6 96.1 mm to (180.3, 66.0)
- moved U10 68.7 mm to (180.3, 78.7)
- moved SW10 54.5 mm to (194.3, 17.8)
- moved R10 53.9 mm to (85.1, 40.6), turned to 180 degrees
- moved D9 52.8 mm to (95.2, 26.7)
- moved R12 52.1 mm to (92.7, 40.6), turned to 180 degrees
- moved D8 49.1 mm to (82.5, 26.7)
- moved SW11 41.5 mm to (194.3, 26.7)
- moved C4 40.1 mm to (129.5, 102.9), turned to 90 degrees
- moved J6 39.8 mm to (88.9, 35.6)
- moved R32 39.2 mm to (177.8, 44.5)
- moved C2 39.0 mm to (121.9, 90.2), turned to 270 degrees
- moved R18 38.4 mm to (113.0, 40.6), turned to 180 degrees
- moved U5 38.2 mm to (133.3, 54.6)
- moved C1 38.1 mm to (128.3, 92.7)
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Routing:
- net (no net): track 0.00 -> 17.8 mm
- net /PT module interface/prb1_rs_btn: track 5.51 -> 0.00 mm
- net Net-(D8-Pad2): track 4.99 -> 0.00 mm
- net /PT module interface/prb1_pwr_btn: track 4.99 -> 0.00 mm
- net +3V3: track 2.35 -> 0.00 mm

Commit message: bug fix
Parts:
- gave numbers to parts that had none: 2
Changed lines of the file:
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@@
     (links 272)
     (no_connects 272)
-    (area 29.814999 12.305 216.565001 123.575)
+    (area 33.234999 12.305 199.885 108.3942)
     (thickness 1.6)
     (drawings 0)
@@
     (tags "resistor 1206")
     (attr smd)
-    (fp_text reference "" (at 0 -1.85 180) (layer F.SilkS)
+    (fp_text reference R47 (at 0 -1.85 180) (layer F.SilkS)
       (effects (font (size 1 1) (thickness 0.15)))
     )
@@
     (tags "SO SOIC 2.54")
     (attr smd)
-    (fp_text reference "" (at 0 -3.5) (layer F.SilkS)
+    (fp_text reference FET1 (at 0 -3.5) (layer F.SilkS)
       (effects (font (size 1 1) (thickness 0.15)))
     )

Commit message: add connections
Routing:
- net GND: track 0.00 -> 811.7 mm, vias 0 -> 3
- net +3V3: track 0.00 -> 411.3 mm, vias 0 -> 4
- net VCC: track 0.00 -> 248.8 mm, vias 0 -> 3
- net /vaisala_rs485_b: track 0.00 -> 238.1 mm, vias 0 -> 5
- net /vaisala_rs485_a: track 0.00 -> 218.4 mm, vias 0 -> 5
- net VEE: track 0.00 -> 175.3 mm
- net /intermodule_rs485_a: track 0.00 -> 126.6 mm, vias 0 -> 2
- net /intermodule_rs485_b: track 0.00 -> 125.8 mm, vias 0 -> 2
- net /Probe module/prb1_v: track 0.00 -> 115.6 mm, vias 0 -> 2
- net /PT module interface/prb1_pwr_btn: track 0.00 -> 111.9 mm, vias 0 -> 2
- net /Probe module/prb2_v: track 0.00 -> 102.8 mm, vias 0 -> 2
- net /PT module interface 2/prb2_rs_btn: track 0.00 -> 100.9 mm, vias 0 -> 3
- net /PT module interface/prb1_rs_btn: track 0.00 -> 99.2 mm, vias 0 -> 3
- net /PT module MCU/prb_btn_pwr_master: track 0.00 -> 98.8 mm, vias 0 -> 2
- net /PT module interface 2/prb2_pwr_btn: track 0.00 -> 97.1 mm, vias 0 -> 3
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
Commit message: make gerbers
Parts:
- added REF**: MountingHole_2.7mm_M2.5_ISO7380_Pad, Mounting_Holes:MountingHole_2.7mm_M2.5_ISO7380_Pad, F.Cu at (97.8, 102.9)
- added REF**: MountingHole_2.7mm_M2.5_ISO7380_Pad, Mounting_Holes:MountingHole_2.7mm_M2.5_ISO7380_Pad, F.Cu at (182.9, 95.2)
- added REF**: MountingHole_2.7mm_M2.5_ISO7380_Pad, Mounting_Holes:MountingHole_2.7mm_M2.5_ISO7380_Pad, F.Cu at (106.7, 71.1)
- added REF**: MountingHole_2.7mm_M2.5_ISO7380_Pad, Mounting_Holes:MountingHole_2.7mm_M2.5_ISO7380_Pad, F.Cu at (90.2, 62.2)
- added REF**: MountingHole_2.7mm_M2.5_ISO7380_Pad, Mounting_Holes:MountingHole_2.7mm_M2.5_ISO7380_Pad, F.Cu at (102.9, 34.3)
- added REF**: MountingHole_2.7mm_M2.5_ISO7380_Pad, Mounting_Holes:MountingHole_2.7mm_M2.5_ISO7380_Pad, F.Cu at (132.1, 34.3)
- added REF**: MountingHole_2.7mm_M2.5_ISO7380_Pad, Mounting_Holes:MountingHole_2.7mm_M2.5_ISO7380_Pad, F.Cu at (160.0, 34.3)
- added REF**: MountingHole_2.7mm_M2.5_ISO7380_Pad, Mounting_Holes:MountingHole_2.7mm_M2.5_ISO7380_Pad, F.Cu at (188.0, 34.3)
- added REF**: MountingHole_2.7mm_M2.5_ISO7380_Pad, Mounting_Holes:MountingHole_2.7mm_M2.5_ISO7380_Pad, F.Cu at (194.3, 59.7)
- added REF**: MountingHole_2.7mm_M2.5_ISO7380_Pad, Mounting_Holes:MountingHole_2.7mm_M2.5_ISO7380_Pad, F.Cu at (193.0, 102.9)
Other:
- board outline added: 124.5 x 96.5 mm
- board text added: "17.8.2017"
- board text added: "PP7 Rev 0.1"
